File: 3 Elektronik/sensor_current_stand/sensor_current_stand/MCU_Sheet.kicad_sch (KiCad schematic)
At the start: 1 part, among them U1 STM32F446RETx

Commit message: разработка
Parts:
- added C5: 20pF, Capacitor_SMD:C_0805_2012Metric_Pad1.18x1.45mm_HandSolder, symbol Device:C
Changed lines of the file:
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@@
     (effects (font (size 1.27 1.27) bold) (justify left bottom))
   )
-  (hierarchical_label "E_U_MUX" (shape bidirectional) (at 267.97 107.95 0) (fields_autoplaced)
+  (hierarchical_label "E_U_MUX" (shape output) (at 267.97 107.95 0) (fields_autoplaced)
     (effects (font (size 1.27 1.27) bold) (justify left))
   )
@@
     (effects (font (size 1.27 1.27) bold) (justify right))
   )
-  (hierarchical_label "U_MCU" (shape bidirectional) (at 38.1 69.85 180) (fields_autoplaced)
+  (hierarchical_label "U_MCU" (shape bidirectional) (at 39.37 60.96 180) (fields_autoplaced)
     (effects (font (size 1.27 1.27) bold) (justify right))
   )
-  (hierarchical_label "MUX_2" (shape bidirectional) (at 266.7 68.58 0) (fields_autoplaced)
+  (hierarchical_label "MUX_2" (shape output) (at 266.7 68.58 0) (fields_autoplaced)
     (effects (font (size 1.27 1.27) bold) (justify left))
   )
-  (hierarchical_label "MUX_3" (shape bidirectional) (at 267.97 74.93 0) (fields_autoplaced)
+  (hierarchical_label "MUX_3" (shape output) (at 267.97 74.93 0) (fields_autoplaced)
     (effects (font (size 1.27 1.27) bold) (justify left))
   )
-  (hierarchical_label "MUX_4" (shape bidirectional) (at 266.7 81.28 0) (fields_autoplaced)
+  (hierarchical_label "MUX_4" (shape output) (at 266.7 81.28 0) (fields_autoplaced)
     (effects (font (size 1.27 1.27) bold) (justify left))
   )
-  (hierarchical_label "MUX_1" (shape bidirectional) (at 266.7 62.23 0) (fields_autoplaced)
+  (hierarchical_label "MUX_1" (shape output) (at 266.7 62.23 0) (fields_autoplaced)
     (effects (font (size 1.27 1.27) bold) (justify left))
   )
+  (symbol (lib_id "Device:C") (at 73.66 106.68 0) (unit 1)
+    (in_bom yes) (on_board yes) (dnp no) (fields_autoplaced)
+    (property "Reference" "C5" (at 77.47 105.41 0)
+      (effects (font (size 1.27 1.27)) (justify left))
+    )
+    (property "Value" "20pF" (at 77.47 107.95 0)
+      (effects (font (size 1.27 1.27)) (justify left))
+    )
+    (property "Footprint" "Capacitor_SMD:C_0805_2012Metric_Pad1.18x1.45mm_HandSolder" (at 74.6252 110.49 0)
+      (effects (font (size 1.27 1.27)) hide)
+    )
+    (property "Datasheet" "~" (at 73.66 106.68 0)
+      (effects (font (size 1.27 1.27)) hide)
+    )
+    (pin "1")
+    (pin "2")
+    (instances
+      (project "sensor_current_stand"
+        (path "/585f0b4a-d927-4562-b364-ee4ef7ff84cf/99bea5c6-1936-4c20-a256-95e65884bae3"
+          (reference "C5") (unit 1)
+        )
+        (path "/585f0b4a-d927-4562-b364-ee4ef7ff84cf/6f1b9f7e-5fef-4a41-8a49-4f41855a9d38"
+          (reference "C11") (unit 1)
+        )
+      )
+    )
+  )
   (symbol (lib_id "MCU_ST_STM32F4:STM32F446RETx") (at 139.7 90.17 0) (unit 1)

Commit message: quarz
Parts:
- added C5: 20pF, Capacitor_SMD:C_0805_2012Metric_Pad1.18x1.45mm_HandSolder, symbol Device:C
- added R1 (x2): 0, Resistor_SMD:R_1206_3216Metric_Pad1.30x1.75mm_HandSolder, symbol Device:R
- added Y1: Crystal, Crystal:Crystal_HC49-U_Vertical, symbol Device:Crystal
Connections:
- net Earth: now reaches C5.1
- net Earth: now also U1.12 (VSSA), U1.18 (VSS), U1.31 (VSS), U1.47 (VSS), U1.63 (VSS), C5.1
- net at C5.2: now also R1.2, Y1.1
- net USB_DM: now reaches U1.44 (PA11)
- net USB_DP: now reaches U1.45 (PA12)
- net at U1.5 (PH0): now also R1.1
- net at U1.6 (PH1): now also R1.1
- new net: C5.2, R1.2, Y1.2
Other:
- moved on the sheet: C5

Commit message: промежуточная версия
надо правильно подключить прошивалку
Parts:
- added C5: 1uF, Capacitor_SMD:C_0805_2012Metric_Pad1.18x1.45mm_HandSolder, symbol Device:C
- added C5: 100nF, Capacitor_SMD:C_0805_2012Metric_Pad1.18x1.45mm_HandSolder, symbol Device:C
- added C5: 2.2uF, Capacitor_SMD:C_0805_2012Metric_Pad1.18x1.45mm_HandSolder, symbol Device:C
- added J8: Conn_02x05_Odd_Even, Connector_IDC:IDC-Header_2x05_P2.54mm_Vertical, symbol Connector_Generic:Conn_02x05_Odd_Even
- added R2: 10k, Resistor_SMD:R_1206_3216Metric_Pad1.30x1.75mm_HandSolder, symbol Device:R
Connections:
- net Earth: now also C5.1, C5.1, C5.1, J8.3 (Pin_3), J8.4 (Pin_4)
- net U_MCU: now also U1.1 (VBAT), U1.13 (VDDA), U1.19 (VDD), U1.32 (VDD), U1.48 (VDD), U1.64 (VDD), C5.2, C5.2, R2.2
- net at U1.30 (VCAP_1): now also C5.2
- net at U1.60 (BOOT0): now also R2.1
- net RST: now reaches U1.7 (NRST)
- net RST: now also J8.1 (Pin_1)
- new net SWCLK: J8.2 (Pin_2)
- new net SWDIO: J8.6 (Pin_6)
- new net SWIM: J8.5 (Pin_5)
- no-connect marks 0 -> 4
Other:
- note added: "3V3"
- note added: "5V"
- moved on the sheet: C5, R1, Y1

Commit message: MCU
Connections:
- net SWCLK is gone; now on net JTCK_SWCLK: J8.2 (Pin_2)
- net SWDIO is gone; now on net JTMS_SWDIO: J8.6 (Pin_6)
- net SWIM is gone; now on net JTDO_SWO: J8.5 (Pin_5)
- net E_U_MUX: now also U1.33 (PB12)
- net MUX_1_E: now also U1.38 (PC7)
- net MUX_1_S0: now also U1.41 (PA8)
- net MUX_1_S1: now also U1.40 (PC9)
- net MUX_1_S2: now also U1.39 (PC8)
- net MUX_2_E: now also U1.34 (PB13)
- net MUX_2_S0: now also U1.37 (PC6)
- net MUX_2_S1: now also U1.36 (PB15)
- net MUX_2_S2: now also U1.35 (PB14)
- net MUX_3_E: now also U1.26 (PB0)
- net MUX_3_S0: now also U1.29 (PB10)
- net MUX_3_S1: now also U1.28 (PB2)
- net MUX_3_S2: now also U1.27 (PB1)
- net MUX_4_E: now also U1.22 (PA6)
- net MUX_4_S0: now also U1.25 (PC5)
- net MUX_4_S1: now also U1.24 (PC4)
- net MUX_4_S2: now also U1.23 (PA7)
- net JTRST: now reaches J8.7 (Pin_7)
- net JTRST: now also U1.56 (PB4)
- net JTDI: now reaches J8.8 (Pin_8)
- net JTDI: now also U1.50 (PA15)
- net JTMS_SWDIO: now reaches U1.46 (PA13)
- net JTCK_SWCLK: now reaches U1.49 (PA14)
- net JTDO_SWO: now reaches U1.55 (PB3)
- no-connect marks 4 -> 2
Other:
- note added: "3V"
- note added: "Все адресные выходы MUX в 0 Все управляющие выходы включения MUX в 0 Управление включения питания MUX в 0, для включения в 1"
- note added: "Уточнить параметры"
- note added: "куда притягивать?"
- note removed: "3V3"
- moved on the sheet: C5
