File: 3 Elektronik/sensor_current_stand/sensor_current_stand/MUX.kicad_sch (KiCad schematic)
At the start: 0 parts

Commit message: разработка
Parts:
- added R1 (x4): 10k, Resistor_SMD:R_1206_3216Metric_Pad1.30x1.75mm_HandSolder, symbol Device:R
- added U4, U5, U6, U7: 74HC4051, Package_SO:TSSOP-16_4.4x5mm_P0.65mm, symbol 74xx:74HC4051
Connections:
- new net: R1.1, U7.16 (VCC), U7.3 (A)
- new net Earth: U4.7 (VEE), U4.8 (GND), U5.7 (VEE), U5.8 (GND), U6.7 (VEE), U6.8 (GND), U7.7 (VEE), U7.8 (GND)
- new net MUX_1_E: R1.2, U4.6 (~{E})
- new net MUX_1_S0: U4.11 (S0)
- new net MUX_1_S1: U4.10 (S1)
- new net MUX_1_S2: U4.9 (S2)
- new net MUX_2_E: R1.2, U5.6 (~{E})
- new net MUX_2_S0: U5.11 (S0)
- new net MUX_2_S1: U5.10 (S1)
- new net MUX_2_S2: U5.9 (S2)
- new net MUX_3_E: R1.2, U6.6 (~{E})
- new net MUX_3_S0: U6.11 (S0)
- new net MUX_3_S1: U6.10 (S1)
- new net MUX_3_S2: U6.9 (S2)
- new net MUX_4_E: R1.2, U7.6 (~{E})
- new net MUX_4_S0: U7.11 (S0)
- new net MUX_4_S1: U7.10 (S1)
- new net MUX_4_S2: U7.9 (S2)
- new net SW_1_1: U4.13 (A0)
- new net SW_1_2: U4.14 (A1)
- new net SW_1_3: U4.15 (A2)
- new net SW_1_4: U4.12 (A3)
- new net SW_1_5: U4.1 (A4)
- new net SW_1_6: U4.5 (A5)
- new net SW_1_7: U4.2 (A6)
- new net SW_1_8: U4.4 (A7)
- new net SW_2_1: U5.13 (A0)
- new net SW_2_2: U5.14 (A1)
- new net SW_2_3: U5.15 (A2)
- new net SW_2_4: U5.12 (A3)
- new net SW_2_5: U5.1 (A4)
- new net SW_2_6: U5.5 (A5)
- new net SW_2_7: U5.2 (A6)
- new net SW_2_8: U5.4 (A7)
- new net SW_3_1: U6.13 (A0)
- new net SW_3_2: U6.14 (A1)
- new net SW_3_3: U6.15 (A2)
- new net SW_3_4: U6.12 (A3)
- new net SW_3_5: U6.1 (A4)
- new net SW_3_6: U6.5 (A5)
- new net SW_3_7: U6.2 (A6)
- new net SW_3_8: U6.4 (A7)
- new net SW_4_1: U7.13 (A0)
- new net SW_4_2: U7.14 (A1)
- new net SW_4_3: U7.15 (A2)
- new net SW_4_4: U7.12 (A3)
- new net SW_4_5: U7.1 (A4)
- new net SW_4_6: U7.5 (A5)
- new net SW_4_7: U7.2 (A6)
- new net SW_4_8: U7.4 (A7)
- new net U_MUX: R1.1, R1.1, R1.1, U4.16 (VCC), U4.3 (A), U5.16 (VCC), U5.3 (A), U6.16 (VCC), U6.3 (A)

Commit message: MUX sheet готово
Connections:
- net U_MUX: now also R1.1, U7.16 (VCC), U7.3 (A)
Other:
- moved on the sheet: R1, U7

Commit message: Группа 1 разведена но не проверена
Parts:
- removed U5: 74HC4051, Package_SO:TSSOP-16_4.4x5mm_P0.65mm, symbol 74xx:74HC4051
- added U7: 74HC4051, Package_SO:TSSOP-16_4.4x5mm_P0.65mm, symbol 74xx:74HC4051
- renumbered U4 to U5, U7 to U8
Connections:
- net Earth: now also U7.7 (VEE), U7.8 (GND)
- net MUX_2_E: now also U7.6 (~{E})
- net MUX_2_S0: now also U7.11 (S0)
- net MUX_2_S1: now also U7.10 (S1)
- net MUX_2_S2: now also U7.9 (S2)
- net SW_2_1: now also U7.13 (A0)
- net SW_2_2: now also U7.14 (A1)
- net SW_2_3: now also U7.15 (A2)
- net SW_2_4: now also U7.12 (A3)
- net SW_2_5: now also U7.1 (A4)
- net SW_2_6: now also U7.5 (A5)
- net SW_2_7: now also U7.2 (A6)
- net SW_2_8: now also U7.4 (A7)
- net U_MUX: now also U7.16 (VCC), U7.3 (A)

Commit message: Kicad 8
Parts:
- renumbered R1 to R10, R1 to R11, R1 to R8, R1 to R9
