File: 3 Elektronik/sensor_current_stand/sensor_current_stand/Switch_G3.kicad_sch (KiCad schematic)
At the start: 1 part, among them J7 DC37_Plug_MountingHoles

Commit message: Version 2
Connections:
- net RED_27V_1_CS17 is gone; now on net 27V_IN: J7.1
- net RED_27V_1_CS18 is gone; now on net 27V_IN: J7.5
- net RED_27V_1_CS19 is gone; now on net 27V_IN: J7.9
- net RED_27V_1_CS20 is gone; now on net 27V_IN: J7.13
- net RED_27V_1_CS21 is gone; now on net 27V_IN: J7.17
- net RED_27V_1_CS22 is gone; now on net 27V_IN: J7.21
- net RED_27V_1_CS23 is gone; now on net 27V_IN: J7.25
- net RED_27V_1_CS24 is gone; now on net 27V_IN: J7.29
- net Earth: no longer J7.10, J7.14, J7.18, J7.2, J7.22, J7.26, J7.30, J7.6
- new net DT3_{17}: J7.2
- new net DT3_{18}: J7.6
- new net DT3_{19}: J7.10
- new net DT3_{20}: J7.14
- new net DT3_{21}: J7.18
- new net DT3_{22}: J7.22
- new net DT3_{23}: J7.26
- new net DT3_{24}: J7.30
Other:
- sheet Switch_MOSFET16 ports: added none; removed 27V_IN
- sheet Switch_MOSFET17 ports: added none; removed 27V_IN
- sheet Switch_MOSFET18 ports: added none; removed 27V_IN
- sheet Switch_MOSFET19 ports: added none; removed 27V_IN
- sheet Switch_MOSFET20 ports: added none; removed 27V_IN
- sheet Switch_MOSFET21 ports: added none; removed 27V_IN
- sheet Switch_MOSFET22 ports: added none; removed 27V_IN
- sheet Switch_MOSFET23 ports: added none; removed 27V_IN
- note added: "Обозначение выводов ДТ-500М Номер вывода Цветовая маркировка Функциональное назначение 1 Красный Напряжение питания 27 В 2 Белый Общий 3 Желтый Аналоговый выход (+) 4 Синий Аналоговый выход (-)"
