File: 3 Elektronik/sensor_current_stand/sensor_current_stand/Switch_MOSFET.kicad_sch (KiCad schematic)
At the start: 4 parts, among them Q1 BSH201

Commit message: прверка на производстве
Parts:
- C5: footprint Capacitor_SMD:C_1206_3216Metric -> Capacitor_SMD:C_0805_2012Metric
Changed lines of the file:
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@@
       (effects (font (size 1.27 1.27)))
     )
-    (property "Footprint" "Capacitor_SMD:C_1206_3216Metric" (at 125.73 69.5452 0)
+    (property "Footprint" "Capacitor_SMD:C_0805_2012Metric" (at 125.73 69.5452 0)
       (effects (font (size 1.27 1.27)) hide)
     )

Commit message: Kicad 8
Parts:
- renumbered C5 to C18, D5 to D6, Q1 to Q2, R1 to R12

Commit message: Version 2
Parts:
- removed C18: 1uF, Capacitor_SMD:C_0805_2012Metric, symbol Device:C
- removed D6: KP-2012MGC, LED_SMD:LED_0805_2012Metric_Pad1.15x1.40mm_HandSolder, symbol Device:LED
- removed Q2: BSH201, Package_TO_SOT_SMD:SOT-23, symbol test:BSH201
- removed R12: 1.5k, Resistor_SMD:R_1206_3216Metric_Pad1.30x1.75mm_HandSolder, symbol Device:R
- added D5: KP-2012MGC, LED_SMD:LED_0805_2012Metric_Pad1.15x1.40mm_HandSolder, symbol Device:LED
- added Q4: BSS138, Package_TO_SOT_SMD:SOT-23, symbol Transistor_FET:BSS138
- added R15: 10k, Resistor_SMD:R_1206_3216Metric_Pad1.30x1.75mm_HandSolder, symbol Device:R
- added R16: 100, Resistor_SMD:R_1206_3216Metric_Pad1.30x1.75mm_HandSolder, symbol Device:R
- added R17: 50, Resistor_SMD:R_1206_3216Metric_Pad1.30x1.75mm_HandSolder, symbol Device:R
Connections:
- net Earth: now also D5.1 (K), Q4.2 (S), R15.2
- net SW_IN: now also R15.1, R16.2
- net SW_OUT: now also Q4.3 (D)
- new net: Q4.1 (G), R16.1, R17.2
- new net: D5.2 (A), R17.1
