File: 3 Elektronik/sensor_current_stand/sensor_current_stand/secondary_supply.kicad_sch (KiCad schematic)
At the start: 2 parts, among them U2 LD3985M33R_SOT23, U3 LD3985M33R_SOT23

Commit message: разработка
Parts:
- added C1, C4, C6, C9: 1uF, Capacitor_SMD:C_0805_2012Metric_Pad1.18x1.45mm_HandSolder, symbol Device:C
- added C10, C3, C5, C7: 100nF, Capacitor_SMD:C_0805_2012Metric_Pad1.18x1.45mm_HandSolder, symbol Device:C
- added C2, C8: 10nF, Capacitor_SMD:C_0805_2012Metric_Pad1.18x1.45mm_HandSolder, symbol Device:C
- added D2 (x2): BAT60A, Diode_SMD:D_SOD-323, symbol Diode:BAT60A
- added D5, D6: LED, LED_SMD:LED_0805_2012Metric_Pad1.15x1.40mm_HandSolder, symbol Device:LED
- added R1 (x2): 51, Resistor_SMD:R_1206_3216Metric_Pad1.30x1.75mm_HandSolder, symbol Device:R
Connections:
- net USB_U: now also U2.1 (VIN), U2.3 (INH), U3.1 (VIN), U3.3 (INH), C1.1, C3.1, C6.1, C7.1
- net Earth: now reaches U3.2 (GND)
- net Earth: now also U2.2 (GND), C1.2, C10.2, C2.2, C3.2, C4.2, C5.2, C6.2, C7.2, C8.2, C9.2, D5.1 (K), D6.1 (K)
- net at U3.4 (BYP): now also C8.1
- net at U3.5 (VOUT): now also C10.1, C9.1, D2.2 (A)
- net at U2.4 (BYP): now also C2.1
- net at U2.5 (VOUT): now also C4.1, C5.1, D2.2 (A)
- new net: D6.2 (A), R1.1
- new net: D5.2 (A), R1.1
- new net +3V0: D2.1 (K), R1.2
- new net U_MUX: D2.1 (K), R1.2
Other:
- note added: "3V"
- note added: "U_MCU"
- note added: "U_MUX"

Commit message: quarz
Changed lines of the file:
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@@
     (effects (font (size 1.27 1.27)) (justify left))
   )
-  (hierarchical_label "USB" (shape bidirectional) (at 30.48 60.96 180) (fields_autoplaced)
+  (hierarchical_label "USB" (shape input) (at 30.48 60.96 180) (fields_autoplaced)
     (effects (font (size 1.27 1.27) bold) (justify right))
   )

Commit message: secondary supply готово
Other:
- note added: "Для USB"
Changed lines of the file:
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@@
     (effects (font (size 1.27 1.27)) (justify left bottom))
   )
-  (text "Питание МК" (at 85.09 64.77 0)
+  (text "Питание МК" (at 85.09 74.93 0)
     (effects (font (size 1.27 1.27) (thickness 0.254) bold) (justify left bottom))
   )
+  (text "Для USB" (at 170.18 92.71 0)
+    (effects (font (size 1.27 1.27) (thickness 0.254) bold) (justify left bottom))
+  )

Commit message: MCU
Connections:
- net USB_U: no longer U3.3 (INH)
- new net E_U_MUX: U3.3 (INH)
Other:
- note added: "Включение питания MUX по команде"
- moved on the sheet: C7
Changed lines of the file:
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@@
 (kicad_sch (version 20230121) (generator eeschema)
   (paper "A4")
-  (junction (at 81.28 139.7) (diameter 0) (color 0 0 0 0)
-  )
   (junction (at 116.84 157.48) (diameter 0) (color 0 0 0 0)
   )
@@
   (junction (at 114.3 83.82) (diameter 0) (color 0 0 0 0)
   )
-  (junction (at 81.28 137.16) (diameter 0) (color 0 0 0 0)
-  )
-  (junction (at 81.28 157.48) (diameter 0) (color 0 0 0 0)
+  (junction (at 73.66 137.16) (diameter 0) (color 0 0 0 0)
+  )
+  (junction (at 73.66 157.48) (diameter 0) (color 0 0 0 0)
   )
   (junction (at 146.05 137.16) (diameter 0) (color 0 0 0 0)
@@
     (stroke (width 0) (type default))
   )
-  (wire (pts (xy 93.98 157.48) (xy 81.28 157.48))
+  (wire (pts (xy 93.98 157.48) (xy 73.66 157.48))
     (stroke (width 0) (type default))
   )
@@
     (stroke (width 0) (type default))
   )
-  (wire (pts (xy 81.28 137.16) (xy 86.36 137.16))
+  (wire (pts (xy 73.66 137.16) (xy 86.36 137.16))
     (stroke (width 0) (type default))
   )
@@
     (stroke (width 0) (type default))
   )
-  (wire (pts (xy 63.5 137.16) (xy 81.28 137.16))
-    (stroke (width 0) (type default))
-  )
-  (wire (pts (xy 81.28 157.48) (xy 63.5 157.48))
-    (stroke (width 0) (type default))
-  )
-  (wire (pts (xy 81.28 137.16) (xy 81.28 139.7))
+  (wire (pts (xy 63.5 137.16) (xy 73.66 137.16))
+    (stroke (width 0) (type default))
+  )
+  (wire (pts (xy 73.66 157.48) (xy 63.5 157.48))
+    (stroke (width 0) (type default))
+  )
+  (wire (pts (xy 73.66 137.16) (xy 73.66 146.05))
     (stroke (width 0) (type default))
   )
@@
     (stroke (width 0) (type default))
   )
-  (wire (pts (xy 81.28 153.67) (xy 81.28 157.48))
+  (wire (pts (xy 73.66 153.67) (xy 73.66 157.48))
     (stroke (width 0) (type default))
   )
@@
     (stroke (width 0) (type default))
   )
+  (wire (pts (xy 83.82 139.7) (xy 86.36 139.7))
+    (stroke (width 0) (type default))
+  )
   (wire (pts (xy 104.14 157.48) (xy 116.84 157.48))
     (stroke (width 0) (type default))
@@
     (stroke (width 0) (type default))
   )
-  (wire (pts (xy 81.28 139.7) (xy 81.28 146.05))
-    (stroke (width 0) (type default))
-  )
   (wire (pts (xy 140.97 83.82) (xy 143.51 83.82))
     (stroke (width 0) (type default))
@@
   )
   (wire (pts (xy 146.05 137.16) (xy 161.29 137.16))
-    (stroke (width 0) (type default))
-  )
-  (wire (pts (xy 86.36 139.7) (xy 81.28 139.7))
     (stroke (width 0) (type default))
   )
@@
     (effects (font (size 1.27 1.27) bold) (justify left bottom))
   )
+  (text "Включение питания MUX по команде" (at 104.14 123.19 0)
+    (effects (font (size 1.27 1.27) (thickness 0.254) bold) (justify left bottom))
+  )
   (text "U_MUX" (at 149.86 137.16 0)
     (effects (font (size 1.27 1.27)) (justify left bottom))
@@
   (hierarchical_label "U_MUX" (shape output) (at 161.29 137.16 0) (fields_autoplaced)
     (effects (font (size 1.27 1.27)) (justify left))
+  )
+  (hierarchical_label "E_U_MUX" (shape input) (at 83.82 139.7 180) (fields_autoplaced)
+    (effects (font (size 1.27 1.27) bold) (justify right))
   )
   (hierarchical_label "U_MCU" (shape output) (at 158.75 83.82 0) (fields_autoplaced)
@@
     )
   )
-  (symbol (lib_id "Device:C") (at 81.28 149.86 0) (unit 1)
+  (symbol (lib_id "Device:C") (at 73.66 149.86 0) (unit 1)
     (in_bom yes) (on_board yes) (dnp no) (fields_autoplaced)
-    (property "Reference" "C7" (at 85.09 148.59 0)
+    (property "Reference" "C7" (at 77.47 148.59 0)
       (effects (font (size 1.27 1.27)) (justify left))
     )
-    (property "Value" "100nF" (at 85.09 151.13 0)
+    (property "Value" "100nF" (at 77.47 151.13 0)
       (effects (font (size 1.27 1.27)) (justify left))
     )
-    (property "Footprint" "Capacitor_SMD:C_0805_2012Metric_Pad1.18x1.45mm_HandSolder" (at 82.2452 153.67 0)
+    (property "Footprint" "Capacitor_SMD:C_0805_2012Metric_Pad1.18x1.45mm_HandSolder" (at 74.6252 153.67 0)
       (effects (font (size 1.27 1.27)) hide)
     )
-    (property "Datasheet" "~" (at 81.28 149.86 0)
+    (property "Datasheet" "~" (at 73.66 149.86 0)
       (effects (font (size 1.27 1.27)) hide)
     )

Commit message: Группа 1 разведена но не проверена
Parts:
- C10: renamed from C4; footprint Capacitor_SMD:C_0805_2012Metric_Pad1.18x1.45mm_HandSolder -> Capacitor_SMD:C_1206_3216Metric
- C11: renamed from C5; footprint Capacitor_SMD:C_0805_2012Metric_Pad1.18x1.45mm_HandSolder -> Capacitor_SMD:C_1206_3216Metric
- C12: renamed from C3; footprint Capacitor_SMD:C_0805_2012Metric_Pad1.18x1.45mm_HandSolder -> Capacitor_SMD:C_1206_3216Metric
- C13: renamed from C6; footprint Capacitor_SMD:C_0805_2012Metric_Pad1.18x1.45mm_HandSolder -> Capacitor_SMD:C_1206_3216Metric
- C14: renamed from C8; footprint Capacitor_SMD:C_0805_2012Metric_Pad1.18x1.45mm_HandSolder -> Capacitor_SMD:C_1206_3216Metric
- C15: renamed from C9; footprint Capacitor_SMD:C_0805_2012Metric_Pad1.18x1.45mm_HandSolder -> Capacitor_SMD:C_1206_3216Metric
- C16: renamed from C10; footprint Capacitor_SMD:C_0805_2012Metric_Pad1.18x1.45mm_HandSolder -> Capacitor_SMD:C_1206_3216Metric
- C17: renamed from C7; footprint Capacitor_SMD:C_0805_2012Metric_Pad1.18x1.45mm_HandSolder -> Capacitor_SMD:C_1206_3216Metric
- C8: renamed from C1; footprint Capacitor_SMD:C_0805_2012Metric_Pad1.18x1.45mm_HandSolder -> Capacitor_SMD:C_1206_3216Metric
- C9: renamed from C2; footprint Capacitor_SMD:C_0805_2012Metric_Pad1.18x1.45mm_HandSolder -> Capacitor_SMD:C_1206_3216Metric
- D2: renamed from D5; value LED -> KP-2012MGC
- D4: renamed from D6; value LED -> KP-2012MGC
- R? (x2): renamed from R1; value 51 -> 43
- renumbered D2 to D?, U2 to U3, U3 to U4
Connections:
- net +3V0 renamed U_MCU
- net USB_U renamed USB_SUPPL
Other:
- note removed: "3V"
- note removed: "U_MCU"
- note removed: "U_MUX"
- note removed: "Расчет электропитания"

Commit message: прверка на производстве
Parts:
- C10, C11, C12, C13, C14, C15, C16, C17, C8, C9: footprint Capacitor_SMD:C_1206_3216Metric -> Capacitor_SMD:C_0805_2012Metric
Changed lines of the file:
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@@
       (effects (font (size 1.27 1.27)) (justify left))
     )
-    (property "Footprint" "Capacitor_SMD:C_1206_3216Metric" (at 74.6252 153.67 0)
+    (property "Footprint" "Capacitor_SMD:C_0805_2012Metric" (at 74.6252 153.67 0)
       (effects (font (size 1.27 1.27)) hide)
     )
@@
       (effects (font (size 1.27 1.27)) (justify left))
     )
-    (property "Footprint" "Capacitor_SMD:C_1206_3216Metric" (at 102.5652 99.06 0)
+    (property "Footprint" "Capacitor_SMD:C_0805_2012Metric" (at 102.5652 99.06 0)
       (effects (font (size 1.27 1.27)) hide)
     )
@@
       (effects (font (size 1.27 1.27)) (justify left))
     )
-    (property "Footprint" "Capacitor_SMD:C_1206_3216Metric" (at 117.8052 152.4 0)
+    (property "Footprint" "Capacitor_SMD:C_0805_2012Metric" (at 117.8052 152.4 0)
       (effects (font (size 1.27 1.27)) hide)
     )
@@
       (effects (font (size 1.27 1.27)) (justify left))
     )
-    (property "Footprint" "Capacitor_SMD:C_1206_3216Metric" (at 79.7052 100.33 0)
+    (property "Footprint" "Capacitor_SMD:C_0805_2012Metric" (at 79.7052 100.33 0)
       (effects (font (size 1.27 1.27)) hide)
     )
@@
       (effects (font (size 1.27 1.27)) (justify left))
     )
-    (property "Footprint" "Capacitor_SMD:C_1206_3216Metric" (at 127.9652 99.06 0)
+    (property "Footprint" "Capacitor_SMD:C_0805_2012Metric" (at 127.9652 99.06 0)
       (effects (font (size 1.27 1.27)) hide)
     )
@@
       (effects (font (size 1.27 1.27)) (justify left))
     )
-    (property "Footprint" "Capacitor_SMD:C_1206_3216Metric" (at 64.4652 149.86 0)
+    (property "Footprint" "Capacitor_SMD:C_0805_2012Metric" (at 64.4652 149.86 0)
       (effects (font (size 1.27 1.27)) hide)
     )
@@
       (effects (font (size 1.27 1.27)) (justify left))
     )
-    (property "Footprint" "Capacitor_SMD:C_1206_3216Metric" (at 115.2652 99.06 0)
+    (property "Footprint" "Capacitor_SMD:C_0805_2012Metric" (at 115.2652 99.06 0)
       (effects (font (size 1.27 1.27)) hide)
     )
@@
       (effects (font (size 1.27 1.27)) (justify left))
     )
-    (property "Footprint" "Capacitor_SMD:C_1206_3216Metric" (at 61.9252 96.52 0)
+    (property "Footprint" "Capacitor_SMD:C_0805_2012Metric" (at 61.9252 96.52 0)
       (effects (font (size 1.27 1.27)) hide)
     )
@@
       (effects (font (size 1.27 1.27)) (justify left))
     )
-    (property "Footprint" "Capacitor_SMD:C_1206_3216Metric" (at 105.1052 152.4 0)
+    (property "Footprint" "Capacitor_SMD:C_0805_2012Metric" (at 105.1052 152.4 0)
       (effects (font (size 1.27 1.27)) hide)
     )
@@
       (effects (font (size 1.27 1.27)) (justify left))
     )
-    (property "Footprint" "Capacitor_SMD:C_1206_3216Metric" (at 130.5052 152.4 0)
-      (effects (font (size 1.27 1.27)) hide)
-    )
+    (property "Footprint" "Capacitor_SMD:C_0805_2012Metric" (at 130.5052 152.4 0)
+      (effects (font (size 1.27 1.27)) hide)
+    )

Commit message: Kicad 8
Parts:
- gave numbers to parts that had none: 4

Commit message: Version 2
Parts:
- removed C13, C15: 1uF, Capacitor_SMD:C_0805_2012Metric, symbol Device:C
- removed C14: 10nF, Capacitor_SMD:C_0805_2012Metric, symbol Device:C
- removed C16, C17: 100nF, Capacitor_SMD:C_0805_2012Metric, symbol Device:C
- removed D4: KP-2012MGC, LED_SMD:LED_0805_2012Metric_Pad1.15x1.40mm_HandSolder, symbol Device:LED
- removed D5: BAT60A, Diode_SMD:D_SOD-323, symbol Diode:BAT60A
- removed R7: 43, Resistor_SMD:R_1206_3216Metric_Pad1.30x1.75mm_HandSolder, symbol Device:R
- removed U4: LD3985M33R_SOT23, Package_TO_SOT_SMD:SOT-23-5, symbol Regulator_Linear:LD3985M33R_SOT23
Other:
- note removed: "Включение питания MUX по команде"
- note removed: "Питание МUX"
