File: 3 Elektronik/sensor_current_stand/sensor_current_stand/sensor_current_stand.kicad_pcb (KiCad board)
At the start: 2 copper layers, 241.8 x 126.5 mm, 174 parts, among them J1 Conn_01x02_Socket, J2 Conn_01x02_Socket, J3 USB_B, J4 Conn_02x05_Odd_Even, J5 DC37_Plug_MountingHoles, J6 DC37_Plug_MountingHoles, J7 DC37_Plug_MountingHoles, J8 DC37_Plug_MountingHoles, Q1 BSH201, Q10 BSH201, Q11 BSH201, Q12 BSH201, Q13 BSH201, Q14 BSH201, Q15 BSH201, Q16 BSH201, Q17 BSH201, Q18 BSH201, Q19 BSH201, Q2 BSH201, Q20 BSH201, Q21 BSH201, Q22 BSH201, Q23 BSH201, Q24 BSH201, Q25 BSH201, Q26 BSH201, Q27 BSH201, Q28 BSH201, Q29 BSH201, Q3 BSH201, Q30 BSH201, Q31 BSH201, Q32 BSH201, Q4 BSH201, Q5 BSH201, Q6 BSH201, Q7 BSH201, Q8 BSH201, Q9 BSH201, U1 USBLC6-2SC6, U2 STM32F446RETx, U3 LD3985M33R_SOT23, U4 LD3985M33R_SOT23, U5 74HC4051, U6 74HC4051, U7 74HC4051, U8 74HC4051, Y1 Crystal

Commit message: трассировка
Parts:
- moved C39 317.7 mm to (193.9, 98.5), turned to 180 degrees
- moved Q23 317.4 mm to (190.5, 103.0), turned to 90 degrees
- moved R33 314.0 mm to (187.4, 98.5)
- moved D27 311.8 mm to (185.9, 103.0), turned to 90 degrees
- moved Q24 304.6 mm to (174.4, 103.1), turned to 90 degrees
- moved C37 301.6 mm to (193.7, 114.1), turned to 180 degrees
- moved D28 299.8 mm to (170.0, 103.1), turned to 90 degrees
- moved Q21 298.2 mm to (190.4, 118.8), turned to 90 degrees
- moved R31 298.1 mm to (187.3, 114.1)
- moved D25 292.5 mm to (185.8, 118.7), turned to 90 degrees
- moved C36 287.6 mm to (162.6, 98.6), turned to 180 degrees
- moved C38 285.0 mm to (147.0, 98.4), turned to 180 degrees
- moved R30 284.0 mm to (156.4, 98.6)
- moved C40 282.0 mm to (177.6, 98.4), turned to 180 degrees
- moved R32 281.5 mm to (140.9, 98.4)
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Routing:
- net /VOLTMETER_OUT_N: track 77.3 -> 311.1 mm
- net /VOLTMETER_OUT_P: track 52.5 -> 210.8 mm
- net /Switch_G2/RED_27V_1_CS13: track 0.00 -> 127.2 mm, vias 0 -> 2
- net /Switch_G4/RED_27V_1_CS29: track 0.00 -> 127.2 mm, vias 0 -> 2
- net /Switch_G3/RED_27V_1_CS21: track 0.00 -> 127.2 mm, vias 0 -> 2
- net /Switch_G4/RED_27V_1_CS26: track 0.00 -> 78.8 mm, vias 0 -> 4
- net /Switch_G2/RED_27V_1_CS10: track 0.00 -> 78.6 mm, vias 0 -> 4
- net /Switch_G3/RED_27V_1_CS18: track 0.00 -> 78.6 mm, vias 0 -> 4
- net /Switch_G4/RED_27V_1_CS25: track 0.00 -> 77.9 mm, vias 0 -> 2
- net /Switch_G3/RED_27V_1_CS17: track 0.00 -> 77.8 mm, vias 0 -> 2
- net /Switch_G2/RED_27V_1_CS9: track 0.00 -> 77.8 mm, vias 0 -> 2
- net /MUX/SW_3_8: track 0.00 -> 77.7 mm, vias 0 -> 2
- net /MUX/SW_2_8: track 0.00 -> 77.7 mm, vias 0 -> 2
- net /MUX/SW_4_8: track 0.00 -> 77.7 mm, vias 0 -> 2
- net /Switch_G3/RED_27V_1_CS19: track 0.00 -> 76.2 mm, vias 0 -> 6
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- added copper zone on F.Cu, net /Switch_G2/RED_27V_1_CS10
- added copper zone on F.Cu, net /Switch_G2/RED_27V_1_CS11
- added copper zone on F.Cu, net /Switch_G2/RED_27V_1_CS12
- added copper zone on F.Cu, net /Switch_G2/RED_27V_1_CS13
- added copper zone on F.Cu, net /Switch_G2/RED_27V_1_CS14
- added copper zone on F.Cu, net /Switch_G2/RED_27V_1_CS15
- added copper zone on F.Cu, net /Switch_G2/RED_27V_1_CS16
- added copper zone on F.Cu, net /Switch_G2/RED_27V_1_CS9
- added copper zone on F.Cu, net /Switch_G3/RED_27V_1_CS18
- added copper zone on F.Cu, net /Switch_G3/RED_27V_1_CS19
- added copper zone on F.Cu, net /Switch_G3/RED_27V_1_CS20
- added copper zone on F.Cu, net /Switch_G3/RED_27V_1_CS21
- added copper zone on F.Cu, net /Switch_G3/RED_27V_1_CS22
- added copper zone on F.Cu, net /Switch_G3/RED_27V_1_CS23
- added copper zone on F.Cu, net /Switch_G3/RED_27V_1_CS24
- added copper zone on F.Cu, net /Switch_G4/RED_27V_1_CS25
- added copper zone on F.Cu, net /Switch_G4/RED_27V_1_CS26
- added copper zone on F.Cu, net /Switch_G4/RED_27V_1_CS27
- added copper zone on F.Cu, net /Switch_G4/RED_27V_1_CS28
- added copper zone on F.Cu, net /Switch_G4/RED_27V_1_CS29
- added copper zone on F.Cu, net /Switch_G4/RED_27V_1_CS30
- added copper zone on F.Cu, net /Switch_G4/RED_27V_1_CS31
- added copper zone on F.Cu, net /Switch_G4/RED_27V_1_CS32
Other:
- board size 241.8 x 126.5 mm -> 225.2 x 126.5 mm
- board text added: "J5"
- board text added: "J6"
- board text added: "locked"
- board text removed: "ДТ 1"
- board text removed: "ДТ 10"
- board text removed: "ДТ 11"
- board text removed: "ДТ 12"
- board text removed: "ДТ 14"
- board text removed: "ДТ 15"
- board text removed: "ДТ 16"
- board text removed: "ДТ 2"
- board text removed: "ДТ 3"
- board text removed: "ДТ 4"
- board text removed: "ДТ 5"
- board text removed: "ДТ 6"
- board text removed: "ДТ 7"
- board text removed: "ДТ 8"
- board text removed: "ДТ 9"

Commit message: трассировка
Connections:
- U2 pad 55: unconnected-(U2-PB3-Pad55) -> JTDO_SWO
Routing:
- net /MCU/MUX_1_S2: track 0.00 -> 28.8 mm, vias 0 -> 2
- net /MCU/MUX_1_S1: track 0.72 -> 28.1 mm, vias 0 -> 2
- net /MCU/MUX_1_S0: track 0.72 -> 27.4 mm, vias 0 -> 2
- net /MCU/MUX_1_E: track 5.60 -> 29.0 mm, vias 0 -> 2

Commit message: прверка на производстве
Parts:
- added H1: MountingHole_Pad, MountingHole:MountingHole_4.3mm_M4_Pad_TopBottom, F.Cu at (56.5, 36.4)
- added H2: MountingHole_Pad, MountingHole:MountingHole_4.3mm_M4_Pad_TopBottom, F.Cu at (270.0, 36.4)
- added H3: MountingHole_Pad, MountingHole:MountingHole_4.3mm_M4_Pad_TopBottom, F.Cu at (270.0, 151.2)
- added H4: MountingHole_Pad, MountingHole:MountingHole_4.3mm_M4_Pad_TopBottom, F.Cu at (56.5, 151.2)
- C1, C10, C11, C12, C13, C14, C15, C16, C17, C18, C19, C2, C20, C21, C22, C23, C24, C25, C26, C27, C28, C29, C30, C31, C32, C33, C34, C35, C36, C37, C38, C39, C40, C41, C42, C43, C44, C45, C46, C47, C48, C8, C9: footprint Capacitor_SMD:C_1206_3216Metric -> Capacitor_SMD:C_0805_2012Metric
- moved J1 20.0 mm to (90.2, 151.7)
- moved J2 11.5 mm to (102.9, 151.7)
- moved C7 2.57 mm to (104.8, 69.2), turned to 180 degrees
- moved C2 0.43 mm to (79.9, 39.3)
- moved J3 0.43 mm to (66.7, 49.4)
- moved C16 0.19 mm to (93.4, 102.3), turned to -90 degrees
- moved C14 0.16 mm to (85.7, 102.0), turned to -90 degrees
- moved C15 0.09 mm to (89.6, 102.3), turned to -90 degrees
Connections:
- J1 pad 1: Earth -> /Switch_G1/27V_IN
- J1 pad 2: /Switch_G1/27V_IN -> Earth
- U2 pad 23: /MCU/MUX_4_S2 -> /MCU/MUX_4_S0
- U2 pad 25: /MCU/MUX_4_S0 -> /MCU/MUX_4_S2
- U2 pad 27: /MCU/MUX_3_S2 -> /MCU/MUX_3_S0
- U2 pad 29: /MCU/MUX_3_S0 -> /MCU/MUX_3_S2
- U2 pad 35: /MCU/MUX_2_S2 -> /MCU/MUX_2_S0
- U2 pad 37: /MCU/MUX_2_S0 -> /MCU/MUX_2_S2
- U2 pad 38: /MCU/MUX_1_E -> unconnected-(U2-PC7-Pad38)
- U2 pad 39: /MCU/MUX_1_S2 -> /MCU/MUX_1_S0
- U2 pad 41: /MCU/MUX_1_S0 -> /MCU/MUX_1_S2
- U2 pad 42: unconnected-(U2-PA9-Pad42) -> /MCU/MUX_1_E
Routing:
- net /Switch_G1/27V_IN: track 0.00 -> 891.8 mm, vias 0 -> 36
- net /VOLTMETER_OUT_N: track 311.1 -> 764.7 mm, vias 0 -> 1
- net /VOLTMETER_OUT_P: track 210.8 -> 648.5 mm
- net /MUX/U_MUX: track 0.00 -> 213.1 mm, vias 0 -> 11
- net /MCU/MUX_4_S2: track 0.00 -> 97.3 mm, vias 0 -> 2
- net /MCU/MUX_4_S1: track 0.72 -> 94.8 mm, vias 0 -> 2
- net /MCU/MUX_4_S0: track 0.72 -> 92.3 mm, vias 0 -> 2
- net /MCU/MUX_4_E: track 5.60 -> 96.1 mm
- net /MCU/MUX_3_S2: track 0.00 -> 66.3 mm, vias 0 -> 2
- net /MCU/MUX_3_S1: track 0.72 -> 63.4 mm, vias 0 -> 2
- net /MCU/MUX_3_S0: track 0.72 -> 60.9 mm, vias 0 -> 2
- net /MCU/E_U_MUX: track 0.00 -> 56.1 mm, vias 0 -> 2
- net /MCU/MUX_3_E: track 5.66 -> 59.0 mm
- net /MCU/MUX_2_S2: track 0.00 -> 46.8 mm, vias 0 -> 2
- net /MCU/MUX_2_S1: track 0.72 -> 42.8 mm, vias 0 -> 2
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- added copper zone on F.Cu, net /MUX/U_MUX
- added copper zone on F.Cu, net /Switch_G1/27V_IN
- added copper zone on F.Cu, net /Switch_G3/RED_27V_1_CS17
- added copper zone on B.Cu, net Earth
- added copper zone on F.Cu, net Earth
- removed copper zone on F.Cu, net /VOLTMETER_OUT_N
- removed copper zone on B.Cu, net /VOLTMETER_OUT_P
Other:
- board size 225.2 x 126.5 mm -> 225 x 126 mm
- board text added: "БП +27 В"
- board text added: "Вольтметр"
- board text removed: "J5"
- board text removed: "J6"

Commit message: Version 2
Parts:
- removed C11, C12, C16, C17: 100nF, Capacitor_SMD:C_0805_2012Metric
- removed C13, C15, C18, C19, C20, C21, C22, C23, C24, C25, C26, C27, C28, C29, C30, C31, C32, C33, C34, C35, C36, C37, C38, C39, C40, C41, C42, C43, C44, C45, C46, C47, C48: 1uF, Capacitor_SMD:C_0805_2012Metric
- removed C14: 10nF, Capacitor_SMD:C_0805_2012Metric
- removed D34, D35, D36: KP-2012MGC, LED_SMD:LED_0805_2012Metric_Pad1.15x1.40mm_HandSolder
- removed R5: 0, Resistor_SMD:R_1206_3216Metric_Pad1.30x1.75mm_HandSolder
- removed R6: 43, Resistor_SMD:R_1206_3216Metric_Pad1.30x1.75mm_HandSolder
- removed U4: LD3985M33R_SOT23, Package_TO_SOT_SMD:SOT-23-5
- removed U5, U6, U7, U8: 74HC4051, Package_SO:TSSOP-16_4.4x5mm_P0.65mm
- added C3: 100nF, Capacitor_SMD:C_0805_2012Metric, F.Cu at (89.3, 55.7)
- added R100: 100, Resistor_SMD:R_1206_3216Metric_Pad1.30x1.75mm_HandSolder, F.Cu at (189.5, 127.5)
- added R101: 50, Resistor_SMD:R_1206_3216Metric_Pad1.30x1.75mm_HandSolder, F.Cu at (196.0, 127.5)
- added R43: 100, Resistor_SMD:R_1206_3216Metric_Pad1.30x1.75mm_HandSolder, F.Cu at (189.5, 65.5)
- added R44: 50, Resistor_SMD:R_1206_3216Metric_Pad1.30x1.75mm_HandSolder, F.Cu at (196.0, 65.5)
- added R45: 10k, Resistor_SMD:R_1206_3216Metric_Pad1.30x1.75mm_HandSolder, F.Cu at (169.0, 85.5)
- added R46: 100, Resistor_SMD:R_1206_3216Metric_Pad1.30x1.75mm_HandSolder, F.Cu at (171.5, 80.0)
- added R47: 50, Resistor_SMD:R_1206_3216Metric_Pad1.30x1.75mm_HandSolder, F.Cu at (178.0, 80.0)
- added R48: 10k, Resistor_SMD:R_1206_3216Metric_Pad1.30x1.75mm_HandSolder, F.Cu at (151.5, 85.5)
- added R49: 100, Resistor_SMD:R_1206_3216Metric_Pad1.30x1.75mm_HandSolder, F.Cu at (154.0, 80.0)
- added R50: 50, Resistor_SMD:R_1206_3216Metric_Pad1.30x1.75mm_HandSolder, F.Cu at (160.5, 80.0)
- added R51: 10k, Resistor_SMD:R_1206_3216Metric_Pad1.30x1.75mm_HandSolder, F.Cu at (134.0, 85.5)
- added R52: 100, Resistor_SMD:R_1206_3216Metric_Pad1.30x1.75mm_HandSolder, F.Cu at (136.5, 80.0)
- added R53: 50, Resistor_SMD:R_1206_3216Metric_Pad1.30x1.75mm_HandSolder, F.Cu at (143.0, 80.0)
- added R54: 10k, Resistor_SMD:R_1206_3216Metric_Pad1.30x1.75mm_HandSolder, F.Cu at (169.0, 71.0)
- added R55: 100, Resistor_SMD:R_1206_3216Metric_Pad1.30x1.75mm_HandSolder, F.Cu at (171.5, 65.5)
- added R56: 50, Resistor_SMD:R_1206_3216Metric_Pad1.30x1.75mm_HandSolder, F.Cu at (178.0, 65.5)
- added R57: 10k, Resistor_SMD:R_1206_3216Metric_Pad1.30x1.75mm_HandSolder, F.Cu at (134.0, 102.0)
- added R58: 100, Resistor_SMD:R_1206_3216Metric_Pad1.30x1.75mm_HandSolder, F.Cu at (136.5, 96.5)
- added R59: 50, Resistor_SMD:R_1206_3216Metric_Pad1.30x1.75mm_HandSolder, F.Cu at (143.0, 96.5)
- added R60: 10k, Resistor_SMD:R_1206_3216Metric_Pad1.30x1.75mm_HandSolder, F.Cu at (151.5, 102.0)
- added R61: 100, Resistor_SMD:R_1206_3216Metric_Pad1.30x1.75mm_HandSolder, F.Cu at (154.0, 96.5)
- added R62: 50, Resistor_SMD:R_1206_3216Metric_Pad1.30x1.75mm_HandSolder, F.Cu at (160.5, 96.5)
- added R63: 10k, Resistor_SMD:R_1206_3216Metric_Pad1.30x1.75mm_HandSolder, F.Cu at (151.5, 116.5)
- added R64: 100, Resistor_SMD:R_1206_3216Metric_Pad1.30x1.75mm_HandSolder, F.Cu at (154.0, 111.0)
- added R65: 50, Resistor_SMD:R_1206_3216Metric_Pad1.30x1.75mm_HandSolder, F.Cu at (160.5, 111.0)
- added R66: 10k, Resistor_SMD:R_1206_3216Metric_Pad1.30x1.75mm_HandSolder, F.Cu at (169.0, 116.5)
- added R67: 100, Resistor_SMD:R_1206_3216Metric_Pad1.30x1.75mm_HandSolder, F.Cu at (171.5, 111.0)
- added R68: 50, Resistor_SMD:R_1206_3216Metric_Pad1.30x1.75mm_HandSolder, F.Cu at (178.0, 111.0)
- added R69: 10k, Resistor_SMD:R_1206_3216Metric_Pad1.30x1.75mm_HandSolder, F.Cu at (169.0, 101.7)
- added R70: 100, Resistor_SMD:R_1206_3216Metric_Pad1.30x1.75mm_HandSolder, F.Cu at (171.5, 96.5)
- added R71: 50, Resistor_SMD:R_1206_3216Metric_Pad1.30x1.75mm_HandSolder, F.Cu at (178.0, 96.5)
- added R72: 10k, Resistor_SMD:R_1206_3216Metric_Pad1.30x1.75mm_HandSolder, F.Cu at (187.0, 116.5)
- added R73: 100, Resistor_SMD:R_1206_3216Metric_Pad1.30x1.75mm_HandSolder, F.Cu at (189.5, 111.0)
- added R74: 50, Resistor_SMD:R_1206_3216Metric_Pad1.30x1.75mm_HandSolder, F.Cu at (196.1, 111.0)
- added R75: 10k, Resistor_SMD:R_1206_3216Metric_Pad1.30x1.75mm_HandSolder, F.Cu at (187.0, 102.0)
- added R76: 100, Resistor_SMD:R_1206_3216Metric_Pad1.30x1.75mm_HandSolder, F.Cu at (189.5, 96.5)
- added R77: 50, Resistor_SMD:R_1206_3216Metric_Pad1.30x1.75mm_HandSolder, F.Cu at (196.0, 96.5)
- added R78: 10k, Resistor_SMD:R_1206_3216Metric_Pad1.30x1.75mm_HandSolder, F.Cu at (134.0, 116.5)
- added R79: 100, Resistor_SMD:R_1206_3216Metric_Pad1.30x1.75mm_HandSolder, F.Cu at (136.5, 111.0)
- added R80: 50, Resistor_SMD:R_1206_3216Metric_Pad1.30x1.75mm_HandSolder, F.Cu at (143.0, 111.0)
- added R81: 10k, Resistor_SMD:R_1206_3216Metric_Pad1.30x1.75mm_HandSolder, F.Cu at (169.0, 147.5)
- added R82: 100, Resistor_SMD:R_1206_3216Metric_Pad1.30x1.75mm_HandSolder, F.Cu at (171.5, 142.0)
- added R83: 50, Resistor_SMD:R_1206_3216Metric_Pad1.30x1.75mm_HandSolder, F.Cu at (178.0, 142.0)
- added R84: 10k, Resistor_SMD:R_1206_3216Metric_Pad1.30x1.75mm_HandSolder, F.Cu at (151.5, 147.5)
- added R85: 100, Resistor_SMD:R_1206_3216Metric_Pad1.30x1.75mm_HandSolder, F.Cu at (154.0, 142.0)
- added R86: 50, Resistor_SMD:R_1206_3216Metric_Pad1.30x1.75mm_HandSolder, F.Cu at (160.5, 142.0)
- added R87: 10k, Resistor_SMD:R_1206_3216Metric_Pad1.30x1.75mm_HandSolder, F.Cu at (169.0, 132.9)
- added R88: 100, Resistor_SMD:R_1206_3216Metric_Pad1.30x1.75mm_HandSolder, F.Cu at (171.5, 127.5)
- added R89: 50, Resistor_SMD:R_1206_3216Metric_Pad1.30x1.75mm_HandSolder, F.Cu at (178.0, 127.5)
- added R90: 10k, Resistor_SMD:R_1206_3216Metric_Pad1.30x1.75mm_HandSolder, F.Cu at (151.5, 133.0)
- added R91: 100, Resistor_SMD:R_1206_3216Metric_Pad1.30x1.75mm_HandSolder, F.Cu at (154.0, 127.5)
- added R92: 50, Resistor_SMD:R_1206_3216Metric_Pad1.30x1.75mm_HandSolder, F.Cu at (160.5, 127.5)
- added R93: 10k, Resistor_SMD:R_1206_3216Metric_Pad1.30x1.75mm_HandSolder, F.Cu at (187.0, 147.5)
- added R94: 100, Resistor_SMD:R_1206_3216Metric_Pad1.30x1.75mm_HandSolder, F.Cu at (189.5, 142.0)
- added R95: 50, Resistor_SMD:R_1206_3216Metric_Pad1.30x1.75mm_HandSolder, F.Cu at (196.0, 142.0)
- added R96: 10k, Resistor_SMD:R_1206_3216Metric_Pad1.30x1.75mm_HandSolder, F.Cu at (134.0, 147.5)
- added R97: 100, Resistor_SMD:R_1206_3216Metric_Pad1.30x1.75mm_HandSolder, F.Cu at (136.5, 142.0)
- added R98: 50, Resistor_SMD:R_1206_3216Metric_Pad1.30x1.75mm_HandSolder, F.Cu at (143.0, 142.0)
- added R99: 10k, Resistor_SMD:R_1206_3216Metric_Pad1.30x1.75mm_HandSolder, F.Cu at (187.0, 133.0)
- C10: value 1uF -> 100uF; footprint Capacitor_SMD:C_0805_2012Metric -> Capacitor_SMD:C_0805_2012Metric_Pad1.18x1.45mm_HandSolder
- C4: value 100uF -> 10nF; footprint Capacitor_SMD:C_0805_2012Metric_Pad1.18x1.45mm_HandSolder -> Capacitor_SMD:C_0805_2012Metric
- C5: value 20pF -> 1uF; footprint Capacitor_SMD:C_0805_2012Metric_Pad1.18x1.45mm_HandSolder -> Capacitor_SMD:C_0805_2012Metric
- C6: value 20pF -> 100nF; footprint Capacitor_SMD:C_0805_2012Metric_Pad1.18x1.45mm_HandSolder -> Capacitor_SMD:C_0805_2012Metric
- C7: value 4.7uF GRM21BR71C475KA73L -> 20pF
- C8: value 1uF -> 20pF; footprint Capacitor_SMD:C_0805_2012Metric -> Capacitor_SMD:C_0805_2012Metric_Pad1.18x1.45mm_HandSolder
- C9: value 10nF -> 4.7uF GRM21BR71C475KA73L; footprint Capacitor_SMD:C_0805_2012Metric -> Capacitor_SMD:C_0805_2012Metric_Pad1.18x1.45mm_HandSolder
- D3, D5: value BAT60A -> KP-2012MGC; footprint Diode_SMD:D_SOD-323 -> LED_SMD:LED_0805_2012Metric_Pad1.15x1.40mm_HandSolder
- J1: value Conn_01x02_Socket -> USB_B; footprint Connector:JWT_A3963_1x02_P3.96mm_Vertical -> Connector_USB:USB_B_Lumberg_2411_02_Horizontal
- J3: value USB_B -> Conn_01x02_Socket; footprint Connector_USB:USB_B_Lumberg_2411_02_Horizontal -> Connector:JWT_A3963_1x02_P3.96mm_Vertical
- Q1, Q10, Q11, Q12, Q13, Q14, Q15, Q16, Q17, Q18, Q19, Q2, Q20, Q21, Q22, Q23, Q24, Q25, Q26, Q27, Q28, Q29, Q3, Q30, Q31, Q32, Q4, Q5, Q6, Q7, Q8, Q9: value BSH201 -> BSS138
- R1: value 1.5k -> 43
- R10, R3: value 10k -> 100
- R11: value 10k -> 50
- R12, R15, R18, R21, R24, R27, R30, R33, R36, R39, R42: value 1.5k -> 10k
- R13, R16, R19, R22, R25, R28, R31, R34, R37, R40: value 1.5k -> 100
- R14, R17, R20, R23, R26, R29, R32, R35, R38, R41: value 1.5k -> 50
- R4: value 0 -> 50
- R7: value 43 -> 10k
- U2: value STM32F446RETx -> LD3985M33R_SOT23; footprint Package_QFP:LQFP-64_10x10mm_P0.5mm -> Package_TO_SOT_SMD:SOT-23-5
- U3: value LD3985M33R_SOT23 -> STM32F446RETx; footprint Package_TO_SOT_SMD:SOT-23-5 -> Package_QFP:LQFP-64_10x10mm_P0.5mm
- moved D4 124.2 mm to (197.5, 39.5), turned to 90 degrees
- moved D1 123.5 mm to (96.0, 50.8), turned to 0 degrees
- moved C1 123.1 mm to (93.0, 55.7), turned to -90 degrees
- moved R1 117.2 mm to (101.6, 50.8)
- moved D3 106.3 mm to (197.5, 85.0), turned to 90 degrees
- moved J3 104.1 mm to (86.9, 151.4), turned to 0 degrees
- moved R11 98.6 mm to (196.0, 80.0), turned to 180 degrees
- moved R4 91.4 mm to (143.0, 127.5)
- moved R38 91.0 mm to (143.0, 65.5), turned to 180 degrees
- moved R3 89.1 mm to (136.5, 127.5)
- moved J1 84.2 mm to (81.7, 68.0), turned to 180 degrees
- moved D2 82.6 mm to (144.5, 132.5), turned to 90 degrees
- moved R28 81.3 mm to (189.5, 49.0), turned to 180 degrees
- moved R2 81.1 mm to (134.0, 133.0), turned to -90 degrees
- moved R40 79.6 mm to (154.0, 65.5), turned to 180 degrees
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Connections:
- C1 pad 1: Earth -> /USB.U
- C1 pad 2: /Switch_G4/RED_27V_1_CS31 -> Earth
- C10 pad 1: Net-(D3-A) -> Earth
- C10 pad 2: Earth -> RST
- C4 pad 1: Earth -> Net-(U2-BYP)
- C4 pad 2: RST -> Earth
- C5 pad 1: Earth -> /MCU/U_MCU
- C5 pad 2: Net-(C5-Pad2) -> Earth
- C6 pad 1: Earth -> /MCU/U_MCU
- C6 pad 2: Net-(C6-Pad2) -> Earth
- C7 pad 2: Net-(U2-VCAP_1) -> Net-(U3-PH0)
- C8 pad 1: /USB.U -> Earth
- C8 pad 2: Earth -> Net-(U3-PH1)
- C9 pad 1: Net-(U3-BYP) -> Earth
- C9 pad 2: Earth -> Net-(U3-VCAP_1)
- D3 pad 1: /MCU/U_MCU -> Earth
- D5 pad 1: /MUX/U_MUX -> Earth
- J1 pad 1: /Switch_G1/27V_IN -> /USB.U
- J1 pad 2: Earth -> /USBD-
- J2 pad 1: /VOLTMETER_OUT_P -> /Switch_G1/27V_IN
- J2 pad 2: /VOLTMETER_OUT_N -> Earth
- J3 pad 1: /USB.U -> /VOLTMETER_OUT_P
- J3 pad 2: /USBD- -> /VOLTMETER_OUT_N
- J4 pad 3: unconnected-(J4-Pin_3-Pad3) -> /MCU/U_MCU
- J5 pad 1: /Switch_G1/RED_27V_1_CS1 -> /Switch_G1/27V_IN
- J5 pad 10: Earth -> /Switch_G1/DT1_{3}
- J5 pad 13: /Switch_G1/RED_27V_1_CS4 -> /Switch_G1/27V_IN
- J5 pad 14: Earth -> /Switch_G1/DT1_{4}
- J5 pad 17: /Switch_G1/RED_27V_1_CS5 -> /Switch_G1/27V_IN
- J5 pad 18: Earth -> /Switch_G1/DT1_{5}
- J5 pad 2: Earth -> /Switch_G1/DT1_{1}
- J5 pad 21: /Switch_G1/RED_27V_1_CS6 -> /Switch_G1/27V_IN
- J5 pad 22: Earth -> /Switch_G1/DT1_{6}
- J5 pad 25: /Switch_G1/RED_27V_1_CS7 -> /Switch_G1/27V_IN
- J5 pad 26: Earth -> /Switch_G1/DT1_{7}
- J5 pad 29: /Switch_G1/RED_27V_1_CS8 -> /Switch_G1/27V_IN
- J5 pad 30: Earth -> /Switch_G1/DT1_{8}
- J5 pad 5: /Switch_G1/RED_27V_1_CS2 -> /Switch_G1/27V_IN
- J5 pad 6: Earth -> /Switch_G1/DT1_{2}
- J5 pad 9: /Switch_G1/RED_27V_1_CS3 -> /Switch_G1/27V_IN
- J6 pad 1: /Switch_G2/RED_27V_1_CS9 -> /Switch_G1/27V_IN
- J6 pad 10: Earth -> /Switch_G2/DT2_{11}
- J6 pad 13: /Switch_G2/RED_27V_1_CS12 -> /Switch_G1/27V_IN
- J6 pad 14: Earth -> /Switch_G2/DT2_{12}
- J6 pad 17: /Switch_G2/RED_27V_1_CS13 -> /Switch_G1/27V_IN
- J6 pad 18: Earth -> /Switch_G2/DT2_{13}
- J6 pad 2: Earth -> /Switch_G2/DT2_{9}
- J6 pad 21: /Switch_G2/RED_27V_1_CS14 -> /Switch_G1/27V_IN
- J6 pad 22: Earth -> /Switch_G2/DT2_{14}
- J6 pad 25: /Switch_G2/RED_27V_1_CS15 -> /Switch_G1/27V_IN
- J6 pad 26: Earth -> /Switch_G2/DT2_{15}
- J6 pad 29: /Switch_G2/RED_27V_1_CS16 -> /Switch_G1/27V_IN
- J6 pad 30: Earth -> /Switch_G2/DT2_{16}
- J6 pad 5: /Switch_G2/RED_27V_1_CS10 -> /Switch_G1/27V_IN
- J6 pad 6: Earth -> /Switch_G2/DT2_{10}
- J6 pad 9: /Switch_G2/RED_27V_1_CS11 -> /Switch_G1/27V_IN
- J7 pad 1: /Switch_G3/RED_27V_1_CS17 -> /Switch_G1/27V_IN
- J7 pad 10: Earth -> /Switch_G3/DT3_{19}
- J7 pad 13: /Switch_G3/RED_27V_1_CS20 -> /Switch_G1/27V_IN
- J7 pad 14: Earth -> /Switch_G3/DT3_{20}
- J7 pad 17: /Switch_G3/RED_27V_1_CS21 -> /Switch_G1/27V_IN
- J7 pad 18: Earth -> /Switch_G3/DT3_{21}
- J7 pad 2: Earth -> /Switch_G3/DT3_{17}
- J7 pad 21: /Switch_G3/RED_27V_1_CS22 -> /Switch_G1/27V_IN
- J7 pad 22: Earth -> /Switch_G3/DT3_{22}
- J7 pad 25: /Switch_G3/RED_27V_1_CS23 -> /Switch_G1/27V_IN
- J7 pad 26: Earth -> /Switch_G3/DT3_{23}
- J7 pad 29: /Switch_G3/RED_27V_1_CS24 -> /Switch_G1/27V_IN
- J7 pad 30: Earth -> /Switch_G3/DT3_{24}
- J7 pad 5: /Switch_G3/RED_27V_1_CS18 -> /Switch_G1/27V_IN
- J7 pad 6: Earth -> /Switch_G3/DT3_{18}
- J7 pad 9: /Switch_G3/RED_27V_1_CS19 -> /Switch_G1/27V_IN
- J8 pad 1: /Switch_G4/RED_27V_1_CS25 -> /Switch_G1/27V_IN
- J8 pad 10: Earth -> /Switch_G4/DT4_{27}
- J8 pad 13: /Switch_G4/RED_27V_1_CS28 -> /Switch_G1/27V_IN
- J8 pad 14: Earth -> /Switch_G4/DT4_{28}
- J8 pad 17: /Switch_G4/RED_27V_1_CS29 -> /Switch_G1/27V_IN
- J8 pad 18: Earth -> /Switch_G4/DT4_{29}
- J8 pad 2: Earth -> /Switch_G4/DT4_{25}
- J8 pad 21: /Switch_G4/RED_27V_1_CS30 -> /Switch_G1/27V_IN
- J8 pad 22: Earth -> /Switch_G4/DT4_{30}
- J8 pad 25: /Switch_G4/RED_27V_1_CS31 -> /Switch_G1/27V_IN
- J8 pad 26: Earth -> /Switch_G4/DT4_{31}
- J8 pad 29: /Switch_G4/RED_27V_1_CS32 -> /Switch_G1/27V_IN
- J8 pad 30: Earth -> /Switch_G4/DT4_{32}
- J8 pad 5: /Switch_G4/RED_27V_1_CS26 -> /Switch_G1/27V_IN
- J8 pad 6: Earth -> /Switch_G4/DT4_{26}
- J8 pad 9: /Switch_G4/RED_27V_1_CS27 -> /Switch_G1/27V_IN
- Q1 pad 1: /MUX/SW_4_7 -> Net-(Q1-G)
- Q1 pad 2: /Switch_G1/27V_IN -> Earth
- Q1 pad 3: /Switch_G4/RED_27V_1_CS31 -> /Switch_G4/DT4_{25}
- Q10 pad 1: /MUX/SW_2_4 -> Net-(Q10-G)
- Q10 pad 2: /Switch_G1/27V_IN -> Earth
- Q10 pad 3: /Switch_G2/RED_27V_1_CS12 -> /Switch_G1/DT1_{7}
- Q11 pad 1: /MUX/SW_2_7 -> Net-(Q11-G)
- Q11 pad 2: /Switch_G1/27V_IN -> Earth
- Q11 pad 3: /Switch_G2/RED_27V_1_CS15 -> /Switch_G2/DT2_{9}
- Q12 pad 1: /MUX/SW_2_8 -> Net-(Q12-G)
- Q12 pad 2: /Switch_G1/27V_IN -> Earth
- Q12 pad 3: /Switch_G2/RED_27V_1_CS16 -> /Switch_G2/DT2_{10}
- Q13 pad 1: /MUX/SW_2_6 -> Net-(Q13-G)
- Q13 pad 2: /Switch_G1/27V_IN -> Earth
- Q13 pad 3: /Switch_G2/RED_27V_1_CS14 -> /Switch_G2/DT2_{12}
- Q14 pad 1: /MUX/SW_2_5 -> Net-(Q14-G)
- Q14 pad 2: /Switch_G1/27V_IN -> Earth
- Q14 pad 3: /Switch_G2/RED_27V_1_CS13 -> /Switch_G2/DT2_{15}
- Q15 pad 1: /MUX/SW_2_2 -> Net-(Q15-G)
- Q15 pad 2: /Switch_G1/27V_IN -> Earth
- Q15 pad 3: /Switch_G2/RED_27V_1_CS10 -> /Switch_G2/DT2_{14}
- Q16 pad 1: /MUX/SW_2_1 -> Net-(Q16-G)
- Q16 pad 2: /Switch_G1/27V_IN -> Earth
- Q16 pad 3: /Switch_G2/RED_27V_1_CS9 -> /Switch_G2/DT2_{13}
- Q17 pad 1: /MUX/SW_2_3 -> Net-(Q17-G)
- Q17 pad 2: /Switch_G1/27V_IN -> Earth
- Q17 pad 3: /Switch_G2/RED_27V_1_CS11 -> /Switch_G2/DT2_{11}
- Q18 pad 1: /MUX/SW_3_5 -> Net-(Q18-G)
- Q18 pad 2: /Switch_G1/27V_IN -> Earth
- Q18 pad 3: /Switch_G3/RED_27V_1_CS21 -> /Switch_G3/DT3_{17}
- Q19 pad 1: /MUX/SW_3_7 -> Net-(Q19-G)
- Q19 pad 2: /Switch_G1/27V_IN -> Earth
- Q19 pad 3: /Switch_G3/RED_27V_1_CS23 -> /Switch_G3/DT3_{18}
- Q2 pad 1: /MUX/SW_1_1 -> Net-(Q2-G)
- Q2 pad 2: /Switch_G1/27V_IN -> Earth
- Q2 pad 3: /Switch_G1/RED_27V_1_CS1 -> /Switch_G2/DT2_{16}
- Q20 pad 1: /MUX/SW_3_2 -> Net-(Q20-G)
- Q20 pad 2: /Switch_G1/27V_IN -> Earth
- Q20 pad 3: /Switch_G3/RED_27V_1_CS18 -> /Switch_G3/DT3_{22}
- Q21 pad 1: /MUX/SW_3_8 -> Net-(Q21-G)
- Q21 pad 2: /Switch_G1/27V_IN -> Earth
- Q21 pad 3: /Switch_G3/RED_27V_1_CS24 -> /Switch_G3/DT3_{23}
- Q22 pad 1: /MUX/SW_3_1 -> Net-(Q22-G)
- Q22 pad 2: /Switch_G1/27V_IN -> Earth
- Q22 pad 3: /Switch_G3/RED_27V_1_CS17 -> /Switch_G3/DT3_{19}
- Q23 pad 1: /MUX/SW_3_4 -> Net-(Q23-G)
- Q23 pad 2: /Switch_G1/27V_IN -> Earth
- Q23 pad 3: /Switch_G3/RED_27V_1_CS20 -> /Switch_G3/DT3_{24}
- Q24 pad 1: /MUX/SW_3_3 -> Net-(Q24-G)
- Q24 pad 2: /Switch_G1/27V_IN -> Earth
- Q24 pad 3: /Switch_G3/RED_27V_1_CS19 -> /Switch_G3/DT3_{20}
- Q25 pad 1: /MUX/SW_3_6 -> Net-(Q25-G)
- Q25 pad 2: /Switch_G1/27V_IN -> Earth
- Q25 pad 3: /Switch_G3/RED_27V_1_CS22 -> /Switch_G3/DT3_{21}
- Q26 pad 1: /MUX/SW_4_5 -> Net-(Q26-G)
- Q26 pad 2: /Switch_G1/27V_IN -> Earth
- Q26 pad 3: /Switch_G4/RED_27V_1_CS29 -> /Switch_G4/DT4_{31}
- Q27 pad 1: /MUX/SW_4_1 -> Net-(Q27-G)
- Q27 pad 2: /Switch_G1/27V_IN -> Earth
- Q27 pad 3: /Switch_G4/RED_27V_1_CS25 -> /Switch_G4/DT4_{30}
- Q28 pad 1: /MUX/SW_4_8 -> Net-(Q28-G)
- Q28 pad 2: /Switch_G1/27V_IN -> Earth
- Q28 pad 3: /Switch_G4/RED_27V_1_CS32 -> /Switch_G4/DT4_{27}
- Q29 pad 1: /MUX/SW_4_3 -> Net-(Q29-G)
- Q29 pad 2: /Switch_G1/27V_IN -> Earth
- Q29 pad 3: /Switch_G4/RED_27V_1_CS27 -> /Switch_G4/DT4_{26}
- Q3 pad 1: /MUX/SW_1_2 -> Net-(Q3-G)
- Q3 pad 2: /Switch_G1/27V_IN -> Earth
- Q3 pad 3: /Switch_G1/RED_27V_1_CS2 -> /Switch_G1/DT1_{4}
- Q30 pad 1: /MUX/SW_4_6 -> Net-(Q30-G)
- Q30 pad 2: /Switch_G1/27V_IN -> Earth
- Q30 pad 3: /Switch_G4/RED_27V_1_CS30 -> /Switch_G4/DT4_{32}
- Q31 pad 1: /MUX/SW_4_2 -> Net-(Q31-G)
- Q31 pad 2: /Switch_G1/27V_IN -> Earth
- Q31 pad 3: /Switch_G4/RED_27V_1_CS26 -> /Switch_G4/DT4_{29}
- Q32 pad 1: /MUX/SW_4_4 -> Net-(Q32-G)
- Q32 pad 2: /Switch_G1/27V_IN -> Earth
- Q32 pad 3: /Switch_G4/RED_27V_1_CS28 -> /Switch_G4/DT4_{28}
- Q4 pad 1: /MUX/SW_1_3 -> Net-(Q4-G)
- Q4 pad 2: /Switch_G1/27V_IN -> Earth
- Q4 pad 3: /Switch_G1/RED_27V_1_CS3 -> /Switch_G1/DT1_{1}
- Q5 pad 1: /MUX/SW_1_4 -> Net-(Q5-G)
- Q5 pad 2: /Switch_G1/27V_IN -> Earth
- Q5 pad 3: /Switch_G1/RED_27V_1_CS4 -> /Switch_G1/DT1_{2}
- Q6 pad 1: /MUX/SW_1_5 -> Net-(Q6-G)
- Q6 pad 2: /Switch_G1/27V_IN -> Earth
- Q6 pad 3: /Switch_G1/RED_27V_1_CS5 -> /Switch_G1/DT1_{3}
- Q7 pad 1: /MUX/SW_1_6 -> Net-(Q7-G)
- Q7 pad 2: /Switch_G1/27V_IN -> Earth
- Q7 pad 3: /Switch_G1/RED_27V_1_CS6 -> /Switch_G1/DT1_{5}
- Q8 pad 1: /MUX/SW_1_7 -> Net-(Q8-G)
- Q8 pad 2: /Switch_G1/27V_IN -> Earth
- Q8 pad 3: /Switch_G1/RED_27V_1_CS7 -> /Switch_G1/DT1_{8}
- Q9 pad 1: /MUX/SW_1_8 -> Net-(Q9-G)
- Q9 pad 2: /Switch_G1/27V_IN -> Earth
- Q9 pad 3: /Switch_G1/RED_27V_1_CS8 -> /Switch_G1/DT1_{6}
- R1 pad 2: /Switch_G4/RED_27V_1_CS31 -> /MCU/U_MCU
- R10 pad 1: /MUX/U_MUX -> Net-(Q2-G)
- R10 pad 2: /MCU/MUX_2_E -> /MCU/SW2_{16}
- R11 pad 1: /MUX/U_MUX -> Net-(D3-A)
- R11 pad 2: /MCU/MUX_4_E -> Net-(Q2-G)
- R12 pad 1: Net-(D6-A) -> /MCU/SW1_{4}
- R12 pad 2: /Switch_G1/RED_27V_1_CS1 -> Earth
- R13 pad 1: Net-(D7-A) -> Net-(Q3-G)
- R13 pad 2: /Switch_G1/RED_27V_1_CS2 -> /MCU/SW1_{4}
- R14 pad 1: Net-(D8-A) -> Net-(D4-A)
- R14 pad 2: /Switch_G1/RED_27V_1_CS3 -> Net-(Q3-G)
- R15 pad 1: Net-(D9-A) -> /MCU/SW1_{1}
- R15 pad 2: /Switch_G1/RED_27V_1_CS4 -> Earth
- R16 pad 1: Net-(D10-A) -> Net-(Q4-G)
- R16 pad 2: /Switch_G1/RED_27V_1_CS5 -> /MCU/SW1_{1}
- R17 pad 1: Net-(D11-A) -> Net-(D5-A)
- R17 pad 2: /Switch_G1/RED_27V_1_CS6 -> Net-(Q4-G)
- R18 pad 1: Net-(D12-A) -> /MCU/SW1_{2}
- R18 pad 2: /Switch_G1/RED_27V_1_CS7 -> Earth
- R19 pad 1: Net-(D13-A) -> Net-(Q5-G)
- R19 pad 2: /Switch_G1/RED_27V_1_CS8 -> /MCU/SW1_{2}
- R2 pad 1: /MCU/U_MCU -> /MCU/SW4_{25}
- R2 pad 2: RST -> Earth
- R20 pad 1: Net-(D14-A) -> Net-(D6-A)
- R20 pad 2: /Switch_G2/RED_27V_1_CS12 -> Net-(Q5-G)
- R21 pad 1: Net-(D15-A) -> /MCU/SW1_{3}
- R21 pad 2: /Switch_G2/RED_27V_1_CS15 -> Earth
- R22 pad 1: Net-(D16-A) -> Net-(Q6-G)
- R22 pad 2: /Switch_G2/RED_27V_1_CS16 -> /MCU/SW1_{3}
- R23 pad 1: Net-(D17-A) -> Net-(D7-A)
- R23 pad 2: /Switch_G2/RED_27V_1_CS14 -> Net-(Q6-G)
- R24 pad 1: Net-(D18-A) -> /MCU/SW1_{5}
- R24 pad 2: /Switch_G2/RED_27V_1_CS13 -> Earth
- R25 pad 1: Net-(D19-A) -> Net-(Q7-G)
- R25 pad 2: /Switch_G2/RED_27V_1_CS10 -> /MCU/SW1_{5}
- R26 pad 1: Net-(D20-A) -> Net-(D8-A)
- R26 pad 2: /Switch_G2/RED_27V_1_CS9 -> Net-(Q7-G)
- R27 pad 1: Net-(D21-A) -> /MCU/SW1_{8}
- R27 pad 2: /Switch_G2/RED_27V_1_CS11 -> Earth
- R28 pad 1: Net-(D22-A) -> Net-(Q8-G)
- R28 pad 2: /Switch_G3/RED_27V_1_CS21 -> /MCU/SW1_{8}
- R29 pad 1: Net-(D23-A) -> Net-(D9-A)
- R29 pad 2: /Switch_G3/RED_27V_1_CS23 -> Net-(Q8-G)
- R3 pad 1: Net-(U2-BOOT0) -> Net-(Q1-G)
- R3 pad 2: /MCU/U_MCU -> /MCU/SW4_{25}
- R30 pad 1: Net-(D24-A) -> /MCU/SW1_{6}
- R30 pad 2: /Switch_G3/RED_27V_1_CS18 -> Earth
- R31 pad 1: Net-(D25-A) -> Net-(Q9-G)
- R31 pad 2: /Switch_G3/RED_27V_1_CS24 -> /MCU/SW1_{6}
- R32 pad 1: Net-(D26-A) -> Net-(D10-A)
- R32 pad 2: /Switch_G3/RED_27V_1_CS17 -> Net-(Q9-G)
- R33 pad 1: Net-(D27-A) -> /MCU/SW1_{7}
- R33 pad 2: /Switch_G3/RED_27V_1_CS20 -> Earth
- R34 pad 1: Net-(D28-A) -> Net-(Q10-G)
- R34 pad 2: /Switch_G3/RED_27V_1_CS19 -> /MCU/SW1_{7}
- R35 pad 1: Net-(D29-A) -> Net-(D11-A)
- R35 pad 2: /Switch_G3/RED_27V_1_CS22 -> Net-(Q10-G)
- R36 pad 1: Net-(D30-A) -> /MCU/SW2_{9}
- R36 pad 2: /Switch_G4/RED_27V_1_CS29 -> Earth
- R37 pad 1: Net-(D31-A) -> Net-(Q11-G)
- R37 pad 2: /Switch_G4/RED_27V_1_CS25 -> /MCU/SW2_{9}
- R38 pad 1: Net-(D32-A) -> Net-(D12-A)
- R38 pad 2: /Switch_G4/RED_27V_1_CS32 -> Net-(Q11-G)
- R39 pad 1: Net-(D33-A) -> /MCU/SW2_{10}
- R39 pad 2: /Switch_G4/RED_27V_1_CS27 -> Earth
- R4 pad 1: Net-(U2-PH0) -> Net-(D2-A)
- R4 pad 2: Net-(C5-Pad2) -> Net-(Q1-G)
- R40 pad 1: Net-(D34-A) -> Net-(Q12-G)
- R40 pad 2: /Switch_G4/RED_27V_1_CS30 -> /MCU/SW2_{10}
- R41 pad 1: Net-(D35-A) -> Net-(D13-A)
- R41 pad 2: /Switch_G4/RED_27V_1_CS26 -> Net-(Q12-G)
- R42 pad 1: Net-(D36-A) -> /MCU/SW2_{12}
- R42 pad 2: /Switch_G4/RED_27V_1_CS28 -> Earth
- R7 pad 1: Net-(D4-A) -> Net-(U3-BOOT0)
- R7 pad 2: /MUX/U_MUX -> Earth
- R8 pad 1: /MUX/U_MUX -> /MCU/U_MCU
- R8 pad 2: /MCU/MUX_1_E -> RST
- R9 pad 1: /MUX/U_MUX -> /MCU/SW2_{16}
- R9 pad 2: /MCU/MUX_3_E -> Earth
- U2 pad 1: /MCU/U_MCU -> /USB.U
- U2 pad 2: unconnected-(U2-PC13-Pad2) -> Earth
- U2 pad 3: unconnected-(U2-PC14-Pad3) -> /USB.U
- U2 pad 4: unconnected-(U2-PC15-Pad4) -> Net-(U2-BYP)
- U2 pad 5: Net-(U2-PH0) -> /MCU/U_MCU
- U3 pad 1: /USB.U -> /MCU/U_MCU
- U3 pad 2: Earth -> unconnected-(U3-PC13-Pad2)
- U3 pad 3: /USB.U -> unconnected-(U3-PC14-Pad3)
- U3 pad 4: Net-(U3-BYP) -> unconnected-(U3-PC15-Pad4)
- U3 pad 5: Net-(D3-A) -> Net-(U3-PH0)
- Y1 pad 1: Net-(C6-Pad2) -> Net-(U3-PH1)
- Y1 pad 2: Net-(C5-Pad2) -> Net-(U3-PH0)
Routing:
- net /MUX/U_MUX: track 213.1 -> 0.00 mm, vias 11 -> 0
- net /MCU/SW4_{32}: track 0.00 -> 137.1 mm
- net /MCU/SW4_{28}: track 0.00 -> 134.8 mm
- net /Switch_G3/DT3_{21}: track 0.00 -> 134.6 mm
- net /Switch_G1/DT1_{5}: track 0.00 -> 134.6 mm
- net /Switch_G4/DT4_{29}: track 0.00 -> 134.6 mm
- net /Switch_G2/DT2_{13}: track 0.00 -> 134.6 mm
- net /Switch_G1/27V_IN: track 891.8 -> 758.8 mm, vias 36 -> 61
- net /Switch_G2/RED_27V_1_CS13: track 127.4 -> 0.00 mm, vias 2 -> 0
- net /Switch_G1/RED_27V_1_CS5: track 127.2 -> 0.00 mm, vias 2 -> 0
- net /Switch_G4/RED_27V_1_CS29: track 127.2 -> 0.00 mm, vias 2 -> 0
- net /Switch_G3/RED_27V_1_CS21: track 127.2 -> 0.00 mm, vias 2 -> 0
- net /MCU/SW4_{31}: track 0.00 -> 124.3 mm
- net /MCU/SW4_{27}: track 0.00 -> 115.9 mm
- net /MCU/SW4_{30}: track 0.00 -> 108.8 mm
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- removed copper zone on B.Cu, net /MCU/U_MCU
- removed copper zone on F.Cu, net /MCU/U_MCU
- removed copper zone on F.Cu, net /MUX/U_MUX
- removed copper zone on F.Cu, net /Switch_G1/27V_IN
- removed copper zone on F.Cu, net /Switch_G1/RED_27V_1_CS1
- removed copper zone on F.Cu, net /Switch_G1/RED_27V_1_CS2
- removed copper zone on F.Cu, net /Switch_G1/RED_27V_1_CS3
- removed copper zone on F.Cu, net /Switch_G1/RED_27V_1_CS4
- removed copper zone on F.Cu, net /Switch_G1/RED_27V_1_CS5
- removed copper zone on F.Cu, net /Switch_G1/RED_27V_1_CS6
- removed copper zone on F.Cu, net /Switch_G1/RED_27V_1_CS7
- removed copper zone on F.Cu, net /Switch_G1/RED_27V_1_CS8
- removed copper zone on F.Cu, net /Switch_G2/RED_27V_1_CS10
- removed copper zone on F.Cu, net /Switch_G2/RED_27V_1_CS11
- removed copper zone on F.Cu, net /Switch_G2/RED_27V_1_CS12
- removed copper zone on F.Cu, net /Switch_G2/RED_27V_1_CS13
- removed copper zone on F.Cu, net /Switch_G2/RED_27V_1_CS14
- removed copper zone on F.Cu, net /Switch_G2/RED_27V_1_CS15
- removed copper zone on F.Cu, net /Switch_G2/RED_27V_1_CS16
- removed copper zone on F.Cu, net /Switch_G2/RED_27V_1_CS9
- removed copper zone on F.Cu, net /Switch_G3/RED_27V_1_CS17
- removed copper zone on F.Cu, net /Switch_G3/RED_27V_1_CS18
- removed copper zone on F.Cu, net /Switch_G3/RED_27V_1_CS19
- removed copper zone on F.Cu, net /Switch_G3/RED_27V_1_CS20
- removed copper zone on F.Cu, net /Switch_G3/RED_27V_1_CS21
- removed copper zone on F.Cu, net /Switch_G3/RED_27V_1_CS22
- removed copper zone on F.Cu, net /Switch_G3/RED_27V_1_CS23
- removed copper zone on F.Cu, net /Switch_G3/RED_27V_1_CS24
- removed copper zone on F.Cu, net /Switch_G4/RED_27V_1_CS25
- removed copper zone on F.Cu, net /Switch_G4/RED_27V_1_CS26
- removed copper zone on F.Cu, net /Switch_G4/RED_27V_1_CS27
- removed copper zone on F.Cu, net /Switch_G4/RED_27V_1_CS28
- removed copper zone on F.Cu, net /Switch_G4/RED_27V_1_CS29
- removed copper zone on F.Cu, net /Switch_G4/RED_27V_1_CS30
- removed copper zone on F.Cu, net /Switch_G4/RED_27V_1_CS31
- removed copper zone on F.Cu, net /Switch_G4/RED_27V_1_CS32
- removed copper zone on F.Cu, net /USB.U
- removed copper zone on F.Cu, net Net-(D3-A)
- removed copper zone on F.Cu, net Net-(D5-A)
Other:
- board size 225 x 126 mm -> 210 x 126 mm
- board text added: "+"
- board text added: "-"
- board text added: "БП ДТ +27 В"
- board text added: "ДТ 1"
- board text added: "ДТ 10"
- board text added: "ДТ 11"
- board text added: "ДТ 12"
- board text added: "ДТ 14"
- board text added: "ДТ 15"
- board text added: "ДТ 16"
- board text added: "ДТ 17"
- board text added: "ДТ 18"
- board text added: "ДТ 19"
- board text added: "ДТ 2"
- board text added: "ДТ 20"
- board text added: "ДТ 21"
- board text added: "ДТ 22"
- board text added: "ДТ 23"
- board text added: "ДТ 24"
- board text added: "ДТ 25"
- board text added: "ДТ 26"
- board text added: "ДТ 27"
- board text added: "ДТ 28"
- board text added: "ДТ 29"
- board text added: "ДТ 3"
- board text added: "ДТ 30"
- board text added: "ДТ 31"
- board text added: "ДТ 32"
- board text added: "ДТ 4"
- board text added: "ДТ 5"
- board text added: "ДТ 6"
- board text added: "ДТ 7"
- board text added: "ДТ 8"
- board text added: "ДТ 9"
- board text removed: "locked"
- board text removed: "БП +27 В"
