File: 3 Elektronik/sensor_current_stand/sensor_current_stand/sensor_current_stand.kicad_sch (KiCad schematic)
At the start: 3 parts, among them J1 Conn_01x02_Socket, J2 Conn_01x02_Socket, J7 USB_B

Commit message: разработка
Parts:
- added D1, D2: BAT60A, Diode_SMD:D_SOD-323, symbol Diode:BAT60A
- added R1, R2: 22, Resistor_SMD:R_1206_3216Metric_Pad1.30x1.75mm_HandSolder, symbol Device:R
- added R3: 1K5, Resistor_SMD:R_1206_3216Metric_Pad1.30x1.75mm_HandSolder, symbol Device:R
Connections:
- net USB_GND is gone; now on net Earth: J7.4 (GND)
- net USB_D_N: now also R2.1; no longer J7.2 (D-)
- net USB_D_P: now also R1.1; no longer J7.3 (D+)
- net USB_U: now also D2.1 (K); no longer J7.1 (VBUS)
- net Switch_Sheet/0V_IN: now reaches J1.1 (Pin_1)
- net Switch_Sheet/27V_IN: now reaches J1.2 (Pin_2)
- net VOLTMETER_OUT_P: now reaches J2.1 (Pin_1)
- net VOLTMETER_OUT_N: now reaches J2.2 (Pin_2)
- net Earth: now reaches J7.5 (Shield)
- new net: J7.2 (D-), R2.2
- new net: D1.1 (K), D2.2 (A)
- new net: D1.2 (A), J7.1 (VBUS)
- new net: J7.3 (D+), R1.2, R3.2
- new net +3V0: R3.1
Other:
- added sheet Switch_Sheet (Switch.kicad_sch)
- sheet Connectors_current_sensor ports: added VOLTMETER_OUT_N, VOLTMETER_OUT_P; removed none
- sheet MUX ports: added MUX_1, MUX_2, MUX_3, MUX_4, SW1, SW2, SW3, SW4, U_MUX; removed none
- sheet secondary_supply_Sheet ports: added U_MCU, U_MUX; removed none
- moved on the sheet: J1, J2, J7

Commit message: quarz
Other:
- sheet MCU_Sheet ports: added E_U_MUX, MUX_1, MUX_2, MUX_3, MUX_4, USB, U_MCU; removed none
- moved on the sheet: J1

Commit message: MCU
Other:
- sheet secondary_supply_Sheet ports: added E_U_MUX; removed none
- note added: "СТАТИКА!"
Changed lines of the file:
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@@
+    (stroke (width 0) (type default))
+  )
+  (wire (pts (xy 132.08 72.39) (xy 132.08 124.46))
     (stroke (width 0) (type default))
   )
@@
     (stroke (width 0) (type default))
   )
+  (wire (pts (xy 132.08 124.46) (xy 76.2 124.46))
+    (stroke (width 0) (type default))
+  )
   (bus (pts (xy 74.93 64.77) (xy 74.93 68.58))
     (stroke (width 0) (type default))
@@
     (stroke (width 0) (type default))
   )
+  (wire (pts (xy 76.2 106.68) (xy 85.09 106.68))
+    (stroke (width 0) (type default))
+  )
   (wire (pts (xy 50.8 60.96) (xy 72.39 60.96))
     (stroke (width 0) (type default))
@@
     (stroke (width 0) (type default))
   )
+  (wire (pts (xy 124.46 72.39) (xy 132.08 72.39))
+    (stroke (width 0) (type default))
+  )
   (wire (pts (xy 26.67 68.58) (xy 43.18 68.58))
+    (stroke (width 0) (type default))
+  )
+  (wire (pts (xy 76.2 124.46) (xy 76.2 106.68))
     (stroke (width 0) (type default))
   )
@@
   (text "Питание +27 в" (at 168.91 33.02 0)
     (effects (font (size 1.27 1.27) (thickness 0.254) bold) (justify left bottom))
+  )
+  (text "СТАТИКА!" (at 34.29 50.8 0)
+    (effects (font (size 1.27 1.27)) (justify left bottom))
   )
   (label "USB_U" (at 59.69 60.96 0) (fields_autoplaced)
@@
       (effects (font (size 1.27 1.27)) (justify left))
     )
+    (pin "E_U_MUX" input (at 85.09 106.68 180)
+      (effects (font (size 1.27 1.27)) (justify left))
+    )

Commit message: Группа 1 разведена но не проверена
Parts:
- removed D1, D2: BAT60A, Diode_SMD:D_SOD-323, symbol Diode:BAT60A
- removed R1, R2: 22, Resistor_SMD:R_1206_3216Metric_Pad1.30x1.75mm_HandSolder, symbol Device:R
- removed R3: 1K5, Resistor_SMD:R_1206_3216Metric_Pad1.30x1.75mm_HandSolder, symbol Device:R
- added C12: 100nF, Capacitor_SMD:C_1206_3216Metric, symbol Device:C
- added U1: USBLC6-2SC6, Package_TO_SOT_SMD:SOT-23-6, symbol Power_Protection:USBLC6-2SC6
- J3: renamed from J7; footprint Connector_USB:USB_A_CNCTech_1001-011-01101_Horizontal -> Connector_USB:USB_B_Lumberg_2411_02_Horizontal
Connections:
- net Switch_G1/0V_IN is gone; now on net Earth: J1.1 (Pin_1)
- net Earth: now also C12.2, U1.2 (GND)
- net USBD-: now reaches J3.2 (D-)
- net USBD-: now also U1.3 (I/O2)
- net USB.U: now reaches J3.1 (VBUS)
- net USB.U: now also C12.1, U1.5 (VBUS)
- net USBD+: now reaches J3.3 (D+)
- net USBD+: now also U1.1 (I/O1)
- new net USB.D+: U1.6 (I/O1)
- new net USB.D-: U1.4 (I/O2)
Other:
- sheet MCU_Sheet renamed MCU
- sheet Switch_Sheet renamed Switch_G1
- sheet secondary_supply_Sheet renamed Secondary_supply
- removed sheet Connectors_current_sensor
- added sheet Switch_G2 (Switch_G2.kicad_sch)
- added sheet Switch_G3 (Switch_G3.kicad_sch)
- added sheet Switch_G4 (Switch_G4.kicad_sch)
- sheet MCU: file MCU_Sheet.kicad_sch -> MCU.kicad_sch
- sheet MCU ports: added USB{D+ D- U}, {MUX_1_S[0..2] MUX_1_E}, {MUX_2_S[0..2] MUX_2_E}, {MUX_3_S[0..2] MUX_3_E}, {MUX_4_S[0..2] MUX_4_E}; removed MUX_1, MUX_2, MUX_3, MUX_4, USB
- sheet MUX ports: added SW_1_[1..8], SW_2_[1..8], SW_3_[1..8], SW_4_[1..8], {MUX_1_S[0..2] MUX_1_E}, {MUX_2_S[0..2] MUX_2_E}, {MUX_3_S[0..2] MUX_3_E}, {MUX_4_S[0..2] MUX_4_E}; removed MUX_1, MUX_2, MUX_3, MUX_4, SW1, SW2, SW3, SW4
- sheet Secondary_supply: file secondary_supply.kicad_sch -> Secondary_supply.kicad_sch
- sheet Secondary_supply ports: added USB_SUPPL; removed USB
- sheet Switch_G1: file Switch.kicad_sch -> Switch_G1.kicad_sch
- sheet Switch_G1 ports: added SW_1_[1..8], VOLTMETER_OUT_N, VOLTMETER_OUT_P; removed 0V_IN
- note added: "27V_IN"
- note added: "Обозначение выводов ДТ-500М Номер вывода Цветовая маркировка Функциональное назначение 1 Красный Напряжение питания 27 В 2 Белый Общий 3 Желтый Аналоговый выход (+) 4 Синий Аналоговый выход (-)"
- note removed: "СТАТИКА!"
- moved on the sheet: J1, J2

Commit message: трассировка
Other:
- moved on the sheet: J1
Changed lines of the file:
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@@
     (stroke (width 0) (type default))
   )
-  (wire (pts (xy 179.07 6.35) (xy 176.53 6.35))
+  (wire (pts (xy 179.07 25.4) (xy 176.53 25.4))
     (stroke (width 0) (type default))
   )
@@
     (stroke (width 0) (type default))
   )
-  (wire (pts (xy 179.07 7.62) (xy 179.07 6.35))
+  (wire (pts (xy 179.07 26.67) (xy 179.07 25.4))
     (stroke (width 0) (type default))
   )
@@
     (stroke (width 0) (type default))
   )
-  (wire (pts (xy 176.53 3.81) (xy 190.5 3.81))
+  (wire (pts (xy 176.53 22.86) (xy 190.5 22.86))
     (stroke (width 0) (type default))
   )
@@
     (stroke (width 0) (type default))
   )
-  (wire (pts (xy 190.5 3.81) (xy 190.5 39.37))
+  (wire (pts (xy 190.5 22.86) (xy 190.5 39.37))
     (stroke (width 0) (type default))
   )
@@
     (stroke (width 0) (type default))
   )
-  (text "27V_IN" (at 182.88 3.81 0)
+  (text "27V_IN" (at 182.88 22.86 0)
     (effects (font (size 1.27 1.27)) (justify left bottom))
   )
@@
     (effects (font (size 1.27 1.27) (thickness 0.254) bold) (justify left bottom))
   )
-  (text "Питание +27 в" (at 166.37 -2.54 0)
+  (text "Питание +27 в" (at 166.37 16.51 0)
     (effects (font (size 1.27 1.27) (thickness 0.254) bold) (justify left bottom))
   )
@@
     (effects (font (size 1.27 1.27) bold) (justify left bottom))
   )
-  (symbol (lib_id "Connector:Conn_01x02_Socket") (at 171.45 6.35 180) (unit 1)
-    (in_bom yes) (on_board yes) (dnp no) (fields_autoplaced)
-    (property "Reference" "J1" (at 172.085 -1.27 0)
+  (symbol (lib_id "Connector:Conn_01x02_Socket") (at 171.45 25.4 180) (unit 1)
+    (in_bom yes) (on_board yes) (dnp no) (fields_autoplaced)
+    (property "Reference" "J1" (at 172.085 17.78 0)
       (effects (font (size 1.27 1.27)))
     )
-    (property "Value" "Conn_01x02_Socket" (at 172.085 1.27 0)
+    (property "Value" "Conn_01x02_Socket" (at 172.085 20.32 0)
       (effects (font (size 1.27 1.27)))
     )
-    (property "Footprint" "Connector:JWT_A3963_1x02_P3.96mm_Vertical" (at 171.45 6.35 0)
-      (effects (font (size 1.27 1.27)) hide)
-    )
-    (property "Datasheet" "~" (at 171.45 6.35 0)
+    (property "Footprint" "Connector:JWT_A3963_1x02_P3.96mm_Vertical" (at 171.45 25.4 0)
+      (effects (font (size 1.27 1.27)) hide)
+    )
+    (property "Datasheet" "~" (at 171.45 25.4 0)
       (effects (font (size 1.27 1.27)) hide)
     )
@@
     )
   )
-  (symbol (lib_id "power:Earth") (at 179.07 7.62 0) (unit 1)
-    (in_bom yes) (on_board yes) (dnp no) (fields_autoplaced)
-    (property "Reference" "#PWR01" (at 179.07 13.97 0)
-      (effects (font (size 1.27 1.27)) hide)
-    )
-    (property "Value" "Earth" (at 179.07 11.43 0)
-      (effects (font (size 1.27 1.27)) hide)
-    )
-    (property "Footprint" "" (at 179.07 7.62 0)
-      (effects (font (size 1.27 1.27)) hide)
-    )
-    (property "Datasheet" "~" (at 179.07 7.62 0)
-      (effects (font (size 1.27 1.27)) hide)
-    )
+  (symbol (lib_id "power:Earth") (at 179.07 26.67 0) (unit 1)
+    (in_bom yes) (on_board yes) (dnp no) (fields_autoplaced)
+    (property "Reference" "#PWR01" (at 179.07 33.02 0)
+      (effects (font (size 1.27 1.27)) hide)
+    )
+    (property "Value" "Earth" (at 179.07 30.48 0)
+      (effects (font (size 1.27 1.27)) hide)
+    )
+    (property "Footprint" "" (at 179.07 26.67 0)
+      (effects (font (size 1.27 1.27)) hide)
+    )
+    (property "Datasheet" "~" (at 179.07 26.67 0)
+      (effects (font (size 1.27 1.27)) hide)
+    )

Commit message: прверка на производстве
Parts:
- added H1, H2, H3, H4: MountingHole_Pad, MountingHole:MountingHole_4.3mm_M4_Pad_TopBottom, symbol Mechanical:MountingHole_Pad
- C12: footprint Capacitor_SMD:C_1206_3216Metric -> Capacitor_SMD:C_0805_2012Metric
Connections:
- net Earth: now also J1.2 (Pin_2), H1.1, H2.1, H3.1, H4.1; no longer J1.1 (Pin_1)
- net Switch_G1/27V_IN: now also J1.1 (Pin_1); no longer J1.2 (Pin_2)
Other:
- moved on the sheet: J1

Commit message: Kicad 8
Parts:
- renumbered C12 to C2

Commit message: Version 2
Parts:
- removed H1: MountingHole_Pad, MountingHole:MountingHole_4.3mm_M4_Pad_TopBottom, symbol Mechanical:MountingHole_Pad
- added C1, C5: 1uF, Capacitor_SMD:C_0805_2012Metric, symbol Device:C
- added C3, C6: 100nF, Capacitor_SMD:C_0805_2012Metric, symbol Device:C
- added C4: 10nF, Capacitor_SMD:C_0805_2012Metric, symbol Device:C
- added D1: KP-2012MGC, LED_SMD:LED_0805_2012Metric_Pad1.15x1.40mm_HandSolder, symbol Device:LED
- added H4: MountingHole_Pad, MountingHole:MountingHole_4.3mm_M4_Pad_TopBottom, symbol Mechanical:MountingHole_Pad
- added R1: 43, Resistor_SMD:R_1206_3216Metric_Pad1.30x1.75mm_HandSolder, symbol Device:R
- added U2: LD3985M33R_SOT23, Package_TO_SOT_SMD:SOT-23-5, symbol Regulator_Linear:LD3985M33R_SOT23
- renumbered H3 to H1, H4 to H3, J3 to J1, J1 to J2, J2 to J3
Connections:
- net Earth: now also C1.2, C3.2, C4.2, C5.2, C6.2, D1.1 (K), H4.1, U2.2 (GND)
- net MCU/U_MCU: now also C5.1, C6.1, R1.2, U2.5 (VOUT)
- net USB.U: now also C1.1, C3.1, U2.1 (VIN), U2.3 (INH)
- new net: D1.2 (A), R1.1
- new net: C4.1, U2.4 (BYP)
Other:
- removed sheet MUX
- removed sheet Secondary_supply
- sheet MCU ports: added SW1_{[1..8]}, SW2_{[9..16]}, SW3_{[17..24]}, SW4_{[25..32]}; removed E_U_MUX, {MUX_1_S[0..2] MUX_1_E}, {MUX_2_S[0..2] MUX_2_E}, {MUX_3_S[0..2] MUX_3_E}, {MUX_4_S[0..2] MUX_4_E}
- sheet Switch_G1 ports: added SW1_{[1..8]}; removed SW_1_[1..8]
- sheet Switch_G2 ports: added SW2_{[9..16]}; removed SW_2_[1..8]
- sheet Switch_G3 ports: added SW3_{[17..24]}; removed SW_3_[1..8]
- sheet Switch_G4 ports: added SW4_{[25..32]}; removed SW_4_[1..8]
- note added: "Питание МК"
- note removed: "Обозначение выводов ДТ-500М Номер вывода Цветовая маркировка Функциональное назначение 1 Красный Напряжение питания 27 В 2 Белый Общий 3 Желтый Аналоговый выход (+) 4 Синий Аналоговый выход (-)"
- moved on the sheet: C2, H1, H3, J1, J2, J3, U1
