File: 3 Elektronik/sensor_current_stand/sensor_current_stand/sensor_current_stand.kicad_sch (KiCad schematic)
At the start: 17 parts, among them J1 USB_B, J2 Conn_01x02_Socket, J3 Conn_01x02_Socket, U1 USBLC6-2SC6, U2 LD3985M33R_SOT23

Commit message: v2 GEREBER
Parts:
- R1: value 43 -> 50
Changed lines of the file:
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@@
 			)
 		)
-		(property "Value" "43"
+		(property "Value" "50"
 			(at 115.57 114.3 90)
 			(effects
