File: 3 Elektronik/sensor_current_stand/sensor_current_stand/MCU.kicad_sch (KiCad schematic)
At the start: 11 parts, among them J8 Conn_02x05_Odd_Even, U1 STM32F446RETx, Y1 Crystal

Commit message: Группа 1 разведена но не проверена
Parts:
- removed C5: 1uF, Capacitor_SMD:C_0805_2012Metric_Pad1.18x1.45mm_HandSolder, symbol Device:C
- removed C5: 100nF, Capacitor_SMD:C_0805_2012Metric_Pad1.18x1.45mm_HandSolder, symbol Device:C
- added C5: 100uF, Capacitor_SMD:C_0805_2012Metric_Pad1.18x1.45mm_HandSolder, symbol Device:C
- added R2: 10k, Resistor_SMD:R_1206_3216Metric_Pad1.30x1.75mm_HandSolder, symbol Device:R
- C5: value 2.2uF -> 4.7uF GRM21BR71C475KA73L
- renumbered J8 to J4
Connections:
- net Earth: now also J4.7 (Pin_7), C5.1; no longer J4.3 (Pin_3), J4.4 (Pin_4)
- net JTDI: now also J4.4 (Pin_4); no longer J4.8 (Pin_8)
- net JTDO_SWO: now also J4.6 (Pin_6); no longer J4.5 (Pin_5), U1.55 (PB3)
- net JTMS_SWDIO: now also J4.1 (Pin_1); no longer J4.6 (Pin_6)
- net JTRST: now also J4.8 (Pin_8); no longer J4.7 (Pin_7)
- net RST: now also J4.5 (Pin_5), C5.2, R2.2; no longer J4.1 (Pin_1)
- net U_MCU: now also R2.1
- net USB_DM renamed USB.D-
- net USB_DP renamed USB.D+
- no-connect marks 2 -> 27
Other:
- note removed: "Уточнить параметры"
- note removed: "куда притягивать?"
- moved on the sheet: J4

Commit message: трассировка
Connections:
- net JTDO_SWO: now also U1.55 (PB3)
Changed lines of the file:
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@@
   (junction (at 90.17 72.39) (diameter 0) (color 0 0 0 0)
   )
+  (junction (at 134.62 38.1) (diameter 0) (color 0 0 0 0)
+  )
   (junction (at 99.06 152.4) (diameter 0) (color 0 0 0 0)
   )
@@
   )
   (junction (at 210.82 33.02) (diameter 0) (color 0 0 0 0)
+  )
+  (junction (at 134.62 22.86) (diameter 0) (color 0 0 0 0)
   )
   (junction (at 144.78 38.1) (diameter 0) (color 0 0 0 0)
@@
     (stroke (width 0) (type default))
   )
-  (wire (pts (xy 102.87 22.86) (xy 142.24 22.86))
+  (wire (pts (xy 102.87 22.86) (xy 134.62 22.86))
     (stroke (width 0) (type default))
   )
@@
     (stroke (width 0) (type default))
   )
+  (wire (pts (xy 157.48 100.33) (xy 162.56 100.33))
+    (stroke (width 0) (type default))
+  )
   (wire (pts (xy 115.57 62.23) (xy 115.57 72.39))
     (stroke (width 0) (type default))
@@
     (stroke (width 0) (type default))
   )
+  (wire (pts (xy 134.62 22.86) (xy 134.62 38.1))
+    (stroke (width 0) (type default))
+  )
   (wire (pts (xy 67.31 59.69) (xy 80.01 59.69))
     (stroke (width 0) (type default))
@@
   )
   (wire (pts (xy 157.48 64.77) (xy 181.61 64.77))
+    (stroke (width 0) (type default))
+  )
+  (wire (pts (xy 134.62 22.86) (xy 142.24 22.86))
     (stroke (width 0) (type default))
   )
@@
       (effects (font (size 1.27 1.27)) (justify left) hide)
     )
+  )
+  (global_label "JTDO_SWO" (shape input) (at 162.56 100.33 0) (fields_autoplaced)
+    (effects (font (size 1.27 1.27)) (justify left))
+    (property "Intersheetrefs" "${INTERSHEET_REFS}" (at 175.0399 100.33 0)
+      (effects (font (size 1.27 1.27)) (justify left) hide)
+    )

Commit message: прверка на производстве
Connections:
- net MUX_1_E: now also U1.42 (PA9); no longer U1.38 (PC7)
- net MUX_1_S0: now also U1.39 (PC8); no longer U1.41 (PA8)
- net MUX_1_S2: now also U1.41 (PA8); no longer U1.39 (PC8)
- net MUX_2_S0: now also U1.35 (PB14); no longer U1.37 (PC6)
- net MUX_2_S2: now also U1.37 (PC6); no longer U1.35 (PB14)
- net MUX_3_S0: now also U1.27 (PB1); no longer U1.29 (PB10)
- net MUX_3_S2: now also U1.29 (PB10); no longer U1.27 (PB1)
- net MUX_4_S0: now also U1.23 (PA7); no longer U1.25 (PC5)
- net MUX_4_S2: now also U1.25 (PC5); no longer U1.23 (PA7)
Changed lines of the file:
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@@
   (junction (at 144.78 38.1) (diameter 0) (color 0 0 0 0)
   )
+  (no_connect (at 121.92 90.17))
   (no_connect (at 121.92 110.49))
   (no_connect (at 157.48 59.69))
-  (no_connect (at 157.48 72.39))
   (no_connect (at 157.48 107.95))
   (no_connect (at 121.92 100.33))
@@
     (stroke (width 0) (type default))
   )
+  (bus_entry (at 176.53 74.93) (size -2.54 -2.54)
+    (stroke (width 0) (type default))
+  )
   (bus_entry (at 181.61 80.01) (size -2.54 -2.54)
     (stroke (width 0) (type default))
@@
     (stroke (width 0) (type default))
   )
-  (bus_entry (at 102.87 92.71) (size 2.54 -2.54)
-    (stroke (width 0) (type default))
-  )
   (bus_entry (at 181.61 82.55) (size -2.54 -2.54)
     (stroke (width 0) (type default))
@@
     (stroke (width 0) (type default))
   )
-  (wire (pts (xy 105.41 90.17) (xy 121.92 90.17))
-    (stroke (width 0) (type default))
-  )
   (bus (pts (xy 205.74 149.86) (xy 95.25 149.86))
     (stroke (width 0) (type default))
@@
     (stroke (width 0) (type default))
   )
+  (bus (pts (xy 176.53 72.39) (xy 176.53 74.93))
+    (stroke (width 0) (type default))
+  )
   (wire (pts (xy 157.48 100.33) (xy 162.56 100.33))
     (stroke (width 0) (type default))
@@
     (stroke (width 0) (type default))
   )
+  (wire (pts (xy 157.48 72.39) (xy 173.99 72.39))
+    (stroke (width 0) (type default))
+  )
   (wire (pts (xy 115.57 128.27) (xy 115.57 123.19))
     (stroke (width 0) (type default))
@@
   )
   (bus (pts (xy 184.15 69.85) (xy 184.15 71.12))
-    (stroke (width 0) (type default))
-  )
-  (bus (pts (xy 102.87 92.71) (xy 102.87 95.25))
     (stroke (width 0) (type default))
   )
@@
     (effects (font (size 1.27 1.27)) (justify left bottom))
   )
-  (label "MUX_2_S0" (at 107.95 87.63 0) (fields_autoplaced)
-    (effects (font (size 1.27 1.27)) (justify left bottom))
-  )
   (label "USB.D+" (at 160.02 80.01 0) (fields_autoplaced)
+    (effects (font (size 1.27 1.27)) (justify left bottom))
+  )
+  (label "MUX_2_S2" (at 107.95 87.63 0) (fields_autoplaced)
+    (effects (font (size 1.27 1.27)) (justify left bottom))
+  )
+  (label "MUX_2_S0" (at 160.02 125.73 0) (fields_autoplaced)
     (effects (font (size 1.27 1.27)) (justify left bottom))
   )
@@
     (effects (font (size 1.27 1.27) bold) (justify left bottom))
   )
-  (label "MUX_3_S2" (at 160.02 95.25 0) (fields_autoplaced)
-    (effects (font (size 1.27 1.27)) (justify left bottom))
-  )
-  (label "MUX_1_E" (at 107.95 90.17 0) (fields_autoplaced)
-    (effects (font (size 1.27 1.27)) (justify left bottom))
-  )
-  (label "MUX_2_S2" (at 160.02 125.73 0) (fields_autoplaced)
+  (label "MUX_3_S0" (at 160.02 95.25 0) (fields_autoplaced)
     (effects (font (size 1.27 1.27)) (justify left bottom))
   )
@@
     (effects (font (size 1.27 1.27) bold) (justify left bottom))
   )
-  (label "MUX_3_S0" (at 160.02 118.11 0) (fields_autoplaced)
+  (label "MUX_3_S2" (at 160.02 118.11 0) (fields_autoplaced)
     (effects (font (size 1.27 1.27)) (justify left bottom))
   )
@@
     (effects (font (size 1.27 1.27)) (justify left bottom))
   )
+  (label "MUX_1_E" (at 160.02 72.39 0) (fields_autoplaced)
+    (effects (font (size 1.27 1.27)) (justify left bottom))
+  )
   (label "MUX_2_E" (at 160.02 123.19 0) (fields_autoplaced)
     (effects (font (size 1.27 1.27)) (justify left bottom))
@@
     (effects (font (size 1.27 1.27)) (justify left bottom))
   )
-  (label "MUX_4_S0" (at 107.95 85.09 0) (fields_autoplaced)
-    (effects (font (size 1.27 1.27)) (justify left bottom))
-  )
-  (label "MUX_1_S0" (at 160.02 69.85 0) (fields_autoplaced)
-    (effects (font (size 1.27 1.27)) (justify left bottom))
-  )
-  (label "MUX_1_S2" (at 107.95 92.71 0) (fields_autoplaced)
+  (label "MUX_4_S2" (at 107.95 85.09 0) (fields_autoplaced)
+    (effects (font (size 1.27 1.27)) (justify left bottom))
+  )
+  (label "MUX_1_S2" (at 160.02 69.85 0) (fields_autoplaced)
+    (effects (font (size 1.27 1.27)) (justify left bottom))
+  )
+  (label "MUX_1_S0" (at 107.95 92.71 0) (fields_autoplaced)
     (effects (font (size 1.27 1.27)) (justify left bottom))
   )
@@
     (effects (font (size 1.27 1.27)) (justify left bottom))
   )
-  (label "MUX_4_S2" (at 160.02 67.31 0) (fields_autoplaced)
-    (effects (font (size 1.27 1.27)) (justify left bottom))
-  )
+  (label "MUX_4_S0" (at 160.02 67.31 0) (fields_autoplaced)
+    (effects (font (size 1.27 1.27)) (justify left bottom))
+  )

Commit message: Kicad 8
Parts:
- renumbered C5 to C4, C5 to C6, C5 to C7, R2 to R3, R1 to R4, R1 to R5, U1 to U2

Commit message: Version 2
Parts:
- removed R4, R5: 0, Resistor_SMD:R_1206_3216Metric_Pad1.30x1.75mm_HandSolder, symbol Device:R
- renumbered C4 to C10, C5 to C7, C6 to C8, C7 to C9, R3 to R7, R2 to R8, U2 to U3
Connections:
- net Earth: now also R7.2
- net U_MCU: now also J4.3 (Pin_3); no longer R7.2
- net at C8.2, Y1.1: now also U3.6 (PH1)
- net at C7.2, Y1.2: now also U3.5 (PH0)
- net SW4_{29}: now reaches U3.14 (PA0)
- net SW4_{30}: now reaches U3.15 (PA1)
- net SW4_{31}: now reaches U3.16 (PA2)
- net SW4_{32}: now reaches U3.17 (PA3)
- net SW4_{28}: now reaches U3.20 (PA4)
- net SW4_{27}: now reaches U3.21 (PA5)
- net SW2_{15}: now reaches U3.38 (PC7)
- net SW2_{9}: now reaches U3.43 (PA10)
- net SW1_{6}: now reaches U3.51 (PC10)
- net SW1_{7}: now reaches U3.52 (PC11)
- net SW1_{8}: now reaches U3.53 (PC12)
- net SW1_{5}: now reaches U3.57 (PB5)
- net SW1_{4}: now reaches U3.58 (PB6)
- net SW1_{3}: now reaches U3.59 (PB7)
- net SW1_{2}: now reaches U3.61 (PB8)
- net SW1_{1}: now reaches U3.62 (PB9)
- net E_U_MUX renamed SW3_{19}
- net MUX_1_E renamed SW2_{10}
- net MUX_1_S0 renamed SW2_{16}
- net MUX_1_S1 renamed SW2_{12}
- net MUX_1_S2 renamed SW2_{11}
- net MUX_2_E renamed SW3_{18}
- net MUX_2_S0 renamed SW3_{17}
- net MUX_2_S1 renamed SW2_{13}
- net MUX_2_S2 renamed SW2_{14}
- net MUX_3_E: no longer names the net of U3.26 (PB0)
- net MUX_3_S0 renamed SW3_{23}
- net MUX_3_S1 renamed SW3_{24}
- net MUX_3_S2 renamed SW3_{20}
- net MUX_4_E renamed SW4_{26}
- net MUX_4_S0 renamed SW4_{25}
- net MUX_4_S1 renamed SW3_{21}
- net MUX_4_S2 renamed SW3_{22}
- no-connect marks 27 -> 11
Other:
- note removed: "3V"
- note removed: "5V"
- note removed: "Все адресные выходы MUX в 0 Все управляющие выходы включения MUX в 0 Управление включения питания MUX в 0, для включения в 1"
- moved on the sheet: C10, J4, R8
